File: hardware/new_babyCadence_Payload/new_babyCadence_Payload.kicad_sch (KiCad schematic)
At the start: 32 parts, among them IC2 MICROFJ-60035-TSV-TR1, J1 Conn_01x05_Female, J2 Conn_01x03_Socket, U1 LT3461ES6#TRPBF, U2 LT1807IS8#PBF, U3 ADS1115IDGS

Commit message: Add files via upload
Parts:
- removed IC2: MICROFJ-60035-TSV-TR1, MICROFJ60035TSVTR1, symbol SiPM:MICROFJ-60035-TSV-TR1
- added D3: MICROFJ-60035-TSV-TR1, 1my_footprints:BGA36C100P6X6_613X613X67, symbol MICROFJ-60035-TSV-TR1:MICROFJ-60035-TSV-TR1
- added J3, J4, J7, J8: Conn_01x01_Pin, MountingHole:MountingHole_2.7mm_M2.5_ISO7380_Pad, symbol Connector:Conn_01x01_Pin
Connections:
- net +5V: now also D3.A1 (CATHODE_1), D3.F6 (CATHODE_2)
- net Anode OUT: now also D3.C1 (ANODE_1), D3.D1 (ANODE_2)
- net GND: now also D3.A2 (NC_1), D3.A3 (NC_2), D3.A4 (NC_3), D3.A5 (NC_4), D3.A6 (NC_5), D3.B1 (NC_6), D3.B2 (NC_7), D3.B3 (NC_8), D3.B4 (NC_9), D3.B5 (NC_10), D3.B6 (NC_11), D3.C2 (NC_12), D3.C3 (NC_13), D3.C4 (NC_14), D3.C5 (NC_15), D3.D2 (NC_16), D3.D3 (NC_17), D3.D4 (NC_18), D3.D5 (NC_19), D3.E1 (NC_20), D3.E2 (NC_21), D3.E3 (NC_22), D3.E4 (NC_23), D3.E5 (NC_24), D3.E6 (NC_25), D3.F1 (NC_26), D3.F2 (NC_27), D3.F3 (NC_28), D3.F4 (NC_29), D3.F5 (NC_30), J3.1 (Pin_1), J4.1 (Pin_1), J7.1 (Pin_1), J8.1 (Pin_1)
Other:
- note added: "12V Out"
- note added: "Analog Out"
- note added: "Cathode Out"
- moved on the sheet: J1
