File: hardware/Baby CADENCE - Cosmic Watch PCB/Cosmic_Watch/Cosmic_Watch.kicad_sch (KiCad schematic)
At the start: 5 parts, among them J1 Conn_Coaxial, J2 Conn_01x02_Pin, U1 Opamp_Dual, U2 LT3461ES6-TRPBF

Commit message: Comments/Reminders
Parts:
- removed D1: MICROFJ-60035-TSV-TR1, MICROFJ60035TSVTR1, symbol SiPM:MICROFJ-60035-TSV-TR1
- removed J1: Conn_Coaxial, symbol Connector:Conn_Coaxial
- removed J2: Conn_01x02_Pin, symbol Connector:Conn_01x02_Pin
- removed U1: Opamp_Dual, symbol Device:Opamp_Dual
- removed U2: LT3461ES6-TRPBF, symbol LT3461:LT3461ES6-TRPBF
Other:
- added sheet Power (power.kicad_sch)
- added sheet Signal Processing (signalprocessing.kicad_sch)
- added sheet Silicon Photomultiplier (SiPM.kicad_sch)
- note removed: "ADS1115 Analog to Digital Converter (ADC)"
- note removed: "LT1807"
- note removed: "LT3461"
- note removed: "SiPM"
- note removed: "Signal Out"
- note removed: "Standalone ADC Output (I2C)"
