File: hardware/Muon PCB/power.kicad_sch (KiCad schematic)
At the start: 10 parts, among them J12 USB_B_Micro, U4 BD33FC0FP

Commit message: uploaded latest progress on pcb layout
updated capacitor footprints, still need to find resistor footprints. started layout
Parts:
- removed U4: BD33FC0FP, Package_TO_SOT_SMD:TO-252-2, symbol Regulator_Linear:BD33FC0FP
- added C22: 10u, Capacitor_SMD:C_0805_2012Metric, symbol Device:C
- added U2: NCP1117-3.3_SOT223, Package_TO_SOT_SMD:SOT-223-3_TabPin2, symbol Regulator_Linear:NCP1117-3.3_SOT223
- C23: renamed from C40; footprint Capacitor_SMD:C_0402_1005Metric -> Capacitor_SMD:C_0805_2012Metric
- C24: renamed from C43; footprint Capacitor_SMD:C_0402_1005Metric -> Capacitor_SMD:C_0805_2012Metric
- D3, D5: footprint LED_SMD:LED_0603_1608Metric -> LED_SMD:LED_0402_1005Metric
- renumbered R19 to R18, R20 to R19
Connections:
- net +3.3V: now also U2.2 (VO)
- net GND: now also C22.2, U2.1 (GND)
- net VBUS: now also J12.1 (VBUS), C22.1, U2.3 (VI)
