File: hardware/Muon PCB/rp2040.kicad_sch (KiCad schematic)
At the start: 31 parts, among them J4 Micro_SD_Card_Det1, J5 Conn_01x02_Pin, SW4 SW_Push_Shielded, SW5 SW_Push_Shielded, U12 RP2040, U3 W25Q128JVS, Y3 ABM8-272-T3

Commit message: uploaded latest progress on pcb layout
updated capacitor footprints, still need to find resistor footprints. started layout
Parts:
- added C15: 10u, Capacitor_SMD:C_0805_2012Metric, symbol Device:C
- added R10, R11: 10k, Resistor_SMD:R_0402_1005Metric, symbol Device:R
- added R8, R9: 5k, Resistor_SMD:R_0402_1005Metric, symbol Device:R
- C1: renamed from C11; footprint Capacitor_SMD:C_0402_1005Metric -> Capacitor_SMD:C_0603_1608Metric
- C12: renamed from C9; footprint Capacitor_SMD:C_0402_1005Metric -> Capacitor_SMD:C_0201_0603Metric
- C13: renamed from C10; footprint Capacitor_SMD:C_0402_1005Metric -> Capacitor_SMD:C_0201_0603Metric
- C2: renamed from C39; footprint Capacitor_SMD:C_0402_1005Metric -> Capacitor_SMD:C_0603_1608Metric
- J5: footprint (none) -> Connector_PinHeader_1.00mm:PinHeader_1x02_P1.00mm_Vertical
- renumbered C37 to C10, C38 to C11, C6 to C14, C18 to C3, C31 to C4, C32 to C5, C33 to C6, C34 to C7, C35 to C8, C36 to C9, R16 to R2, R17 to R3, R23 to R4, R15 to R5, R3 to R6, R5 to R7
Connections:
- net +3.3V: now also C15.1, R10.1, R11.1, R8.1, R9.1
- net GND: now also C15.2
- net GPS Reset: now also U12.30 (GPIO19); no longer U12.15 (GPIO12)
- net SCL0: now also R9.2
- net SCL1: now also R11.2
- net SDA0: now also R8.2
- net SDA1: now also R10.2
Other:
- note added: "(place close to VDD pin)"
- note added: "GPS UART Rx receives from GPS module GPS UART Tx transmits from GPS module"
- note added: "I2C0: Temperature Sensor utilizing 5k pullup resistors I2C1: Power Monitor using 10k pullup resistors"
- note added: "Place I2C pullup resistors close to master device"
- note removed: "(old note from william)"
- note removed: "(william's note)"
- note removed: "I2C0: Temperature Sensor utilizing 5k pullup resistors I2C1: Everything else using 10k pullup resistors"
- note removed: "look at what adafruit module uses: hc4050 buffer"
- note removed: "look into buffer for sd card (SD card on proves kit pcb doesn't work)"
- note removed: "look into if 12MHz will impact data processing of the cosmic watch data which is usually at 16HMz"
- note removed: "microsd data lines can be directly connected to mcu. data lines must be right next to each other in gpio pins (ex: 22-25)"
- note removed: "to my knowledge, alert pins can be connected to any of the GPIO pins"
