File: hardware/Muon PCB/sensors.kicad_sch (KiCad schematic)
At the start: 21 parts, among them J2 Conn_Coaxial, J6 Conn_Coaxial, U1 CD-PA1616D, U13 INA219AxD, U15 TMP1075DSG, U16 RFM98PW

Commit message: uploaded latest progress on pcb layout
updated capacitor footprints, still need to find resistor footprints. started layout
Parts:
- removed FB1: FerriteBead, symbol Device:FerriteBead
- removed R24, R25: 5k, Resistor_SMD:R_0402_1005Metric, symbol Device:R
- added BT1: 3V, Battery:BatteryHolder_Keystone_1058_1x2032, symbol Device:Battery
- added C21: 1uF, Capacitor_SMD:C_0603_1608Metric, symbol Device:C
- added FL1: BLM18BD601SN1J, 1my_footprints:BEADC1608X95N, symbol BLM18BD601SN1J:BLM18BD601SN1J
- added R13: 10k, Resistor_SMD:R_0402_1005Metric, symbol Device:R
- C17: renamed from C44; value 0.01uF -> 10nF
- C19: renamed from C20; footprint Capacitor_SMD:C_0402_1005Metric -> Capacitor_SMD:C_0603_1608Metric
- C20: renamed from C21; value 0.1uf -> 100nF
- D2: footprint LED_SMD:LED_0603_1608Metric -> LED_SMD:LED_0402_1005Metric
- R15: renamed from R28; footprint Resistor_SMD:R_0402_1005Metric -> Resistor_SMD:R_0603_1608Metric
- R16: renamed from R30; footprint Resistor_SMD:R_0402_1005Metric -> Resistor_SMD:R_0603_1608Metric
- R17: renamed from R31; footprint Resistor_SMD:R_0402_1005Metric -> Resistor_SMD:R_0603_1608Metric
- renumbered C17 to C16, C42 to C18, R27 to R12, R29 to R14, TP3 to TP1
Connections:
- net +3.3V: now also FL1.2, R13.1
- net GND: now also BT1.2 (-), C21.2
- net RF NSS: now also R13.2
- net at R14.1, TP1.1, U1.1 (VCC): now also FL1.1
- net VBACKUP: now reaches U1.4 (VBACKUP)
- net VBACKUP: now also BT1.1 (+), C21.1
- no-connect marks 10 -> 9
Other:
- note added: "1pps pin provides one electrical pulse per second. Used to synchronize other devices (not needed)"
- note added: "GPS Backup Power Supply"
- note added: "check up on addresses for all the i2c devices"
- note removed: "1pps pin provides one electrical pulse per second. Used to synchronize with other devices."
- note removed: "connect all the digital input output pins to various gpios on MCU"
- note removed: "connect the uart connections to RP2040"
- note removed: "software support is mainly for UART, so change to UART implementation"
- moved on the sheet: C16, C17, C18, C19, C20, D2, J2, J6, R12, R14, R15, R16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
