File: hardware/PROVES_Cosmic_Watch/SiPM.kicad_sch (KiCad schematic)
At the start: 9 parts, among them IC1 MICROFJ-60035-TSV-TR1

Commit message: Updates
Parts:
- removed IC1: MICROFJ-60035-TSV-TR1, MICROFJ60035TSVTR1, symbol SiPM:MICROFJ-60035-TSV-TR1
- added J5: Conn_Coaxial, symbol Connector:Conn_Coaxial
- added TP10: Far Away Test Point, symbol Connector:TestPoint
- added U4: MICROFC-60035-SMT-TR, SiPM-MicroFC60035:OPTO-SMD_4P-MICROFC-60035-SMT-TR, symbol SiPM_MicroFC60035:MICROFC-60035-SMT-TR
Connections:
- net GND: now also J5.2 (Ext)
- net SiPM Signal: now also U4.1 (ANODE)
- net V_Bias: now also J5.1 (In), TP10.1
- net at C11.1, C12.1, C13.1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: now also U4.3 (CATHODE)
Other:
- note added: "Anode"
- note added: "Cathode"
- note added: "V_Bias Coax Connector"
- moved on the sheet: C10, C11, C12, C13, R12, R13, R14, TP5

Commit message: Added Footprints and Started Layout
Parts:
- removed J5: Conn_Coaxial, symbol Connector:Conn_Coaxial
- removed TP10: Far Away Test Point, symbol Connector:TestPoint
- C10, C11, C12, C13: footprint (none) -> Capacitor_SMD:C_0805_2012Metric
- R12, R13, R14: footprint (none) -> Resistor_SMD:R_0805_2012Metric
- TP5: footprint (none) -> TestPoint:TestPoint_Keystone_5000-5004_Miniature
Other:
- note removed: "Anode"
- note removed: "Cathode"
- note removed: "V_Bias Coax Connector"

Commit message: Removed LDO
Parts:
- removed TP5: Raw Signal Test Point, TestPoint:TestPoint_Keystone_5000-5004_Miniature, symbol Connector:TestPoint
Changed lines of the file:
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@@
-	)
-	(junction
-		(at 125.73 76.2)
-		(diameter 0)
-		(color 0 0 0 0)
 	)
 	(junction
@@
 	(wire
 		(pts
-			(xy 125.73 68.58) (xy 125.73 76.2)
-		)
-		(stroke
-			(width 0)
-			(type default)
-		)
-	)
-	(wire
-		(pts
 			(xy 121.92 44.45) (xy 121.92 41.91)
 		)
@@
 	(wire
 		(pts
-			(xy 115.57 76.2) (xy 125.73 76.2)
+			(xy 115.57 76.2) (xy 139.7 76.2)
 		)
 		(stroke
@@
 		(pts
 			(xy 121.92 41.91) (xy 127 41.91)
-		)
-		(stroke
-			(width 0)
-			(type default)
-		)
-	)
-	(wire
-		(pts
-			(xy 125.73 76.2) (xy 139.7 76.2)
 		)
 		(stroke
@@
 					(unit 1)
 				)
-			)
-		)
-	)
-	(symbol
-		(lib_id "Connector:TestPoint")
-		(at 125.73 68.58 0)
-		(unit 1)
-		(exclude_from_sim no)
-		(in_bom yes)
-		(on_board yes)
-		(dnp no)
-		(property "Reference" "TP5"
-			(at 128.27 66.294 0)
-			(effects
-				(font
-					(size 1.27 1.27)
-				)
-				(justify left)
-			)
-		)
-		(property "Value" "Raw Signal Test Point"
-			(at 128.27 69.088 0)
-			(effects
-				(font
-					(size 1.27 1.27)
-				)
-				(justify left)
-			)
-		)
-		(property "Footprint" "TestPoint:TestPoint_Keystone_5000-5004_Miniature"
-			(at 130.81 68.58 0)
-			(effects
-				(font
-					(size 1.27 1.27)
-				)
-				(hide yes)
-			)
-		)
-		(property "Datasheet" "~"
-			(at 130.81 68.58 0)
-			(effects
-				(font
-					(size 1.27 1.27)
-				)
-				(hide yes)
-			)
-		)
-		(property "Description" "test point"
-			(at 125.73 68.58 0)
-			(effects
-				(font
-					(size 1.27 1.27)
-				)
-				(hide yes)
-			)
-		)
-		(pin "1"
-		)
-		(instances
-			(project ""
-				(path "/901a4a81-3d4a-4d59-b0fc-ea1dade1210f/09770208-9a6f-42aa-9b04-6e9dd61abdb1"
-					(reference "TP5")
-					(unit 1)
-				)

Commit message: Layout Updates
Parts:
- added TP5: Bias Voltage, TestPoint:TestPoint_Keystone_5000-5004_Miniature, symbol Connector:TestPoint
Connections:
- net at C11.1, C12.1, C13.1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: now also TP5.1
Changed lines of the file:
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@@
+	)
+	(junction
+		(at 83.82 41.91)
+		(diameter 0)
+		(color 0 0 0 0)
 	)
 	(junction
@@
 	(wire
 		(pts
+			(xy 83.82 41.91) (xy 99.06 41.91)
+		)
+		(stroke
+			(width 0)
+			(type default)
+		)
+	)
+	(wire
+		(pts
 			(xy 132.08 41.91) (xy 137.16 41.91)
 		)
@@
 	(wire
 		(pts
-			(xy 69.85 41.91) (xy 99.06 41.91)
-		)
-		(stroke
-			(width 0)
-			(type default)
-		)
-	)
-	(wire
-		(pts
 			(xy 115.57 85.09) (xy 115.57 88.9)
 		)
@@
 	(wire
 		(pts
+			(xy 69.85 41.91) (xy 83.82 41.91)
+		)
+		(stroke
+			(width 0)
+			(type default)
+		)
+	)
+	(wire
+		(pts
 			(xy 110.49 41.91) (xy 121.92 41.91)
 		)
@@
 		(pts
 			(xy 69.85 46.99) (xy 82.55 46.99)
+		)
+		(stroke
+			(width 0)
+			(type default)
+		)
+	)
+	(wire
+		(pts
+			(xy 83.82 30.48) (xy 83.82 41.91)
 		)
 		(stroke
@@
 			)
 		)
+	)
+	(symbol
+		(lib_id "Connector:TestPoint")
+		(at 83.82 30.48 0)
+		(unit 1)
+		(exclude_from_sim no)
+		(in_bom yes)
+		(on_board yes)
+		(dnp no)
+		(fields_autoplaced yes)
+		(property "Reference" "TP5"
+			(at 86.36 25.9079 0)
+			(effects
+				(font
+					(size 1.27 1.27)
+				)
+				(justify left)
+			)
+		)
+		(property "Value" "Bias Voltage"
+			(at 86.36 28.4479 0)
+			(effects
+				(font
+					(size 1.27 1.27)
+				)
+				(justify left)
+			)
+		)
+		(property "Footprint" "TestPoint:TestPoint_Keystone_5000-5004_Miniature"
+			(at 88.9 30.48 0)
+			(effects
+				(font
+					(size 1.27 1.27)
+				)
+				(hide yes)
+			)
+		)
+		(property "Datasheet" "~"
+			(at 88.9 30.48 0)
+			(effects
+				(font
+					(size 1.27 1.27)
+				)
+				(hide yes)
+			)
+		)
+		(property "Description" "test point"
+			(at 83.82 30.48 0)
+			(effects
+				(font
+					(size 1.27 1.27)
+				)
+				(hide yes)
+			)
+		)
+		(pin "1"
+		)
+		(instances
+			(project ""
+				(path "/901a4a81-3d4a-4d59-b0fc-ea1dade1210f/09770208-9a6f-42aa-9b04-6e9dd61abdb1"
+					(reference "TP5")
+					(unit 1)
+				)
+			)
+		)

Commit message: Layout Updates
Parts:
- TP5: value Bias Voltage -> V+ Bias
Changed lines of the file:
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@@
 			)
 		)
-		(property "Value" "Bias Voltage"
+		(property "Value" "V+ Bias"
 			(at 86.36 28.4479 0)
 			(effects

Commit message: Layout Updates
Parts:
- added H1, H2, H3, H4: MountingHole_Pad, MountingHole:MountingHole_2.7mm_M2.5, symbol Mechanical:MountingHole_Pad
Connections:
- net GND: now also H1.1, H2.1, H3.1, H4.1
