File: hardware/PROVES_Cosmic_Watch/PROVES_Cosmic_Watch.kicad_pcb (KiCad board)
At the start: 4 copper layers, 88 x 94.5 mm, 53 parts, among them J1 USB_B_Micro, J2 DF11, J3 Conn_Coaxial, U2 LT3461ES6-TRPBF, U3 LT1807, U4 MICROFC-60035-SMT-TR

Commit message: Updates
Parts:
- moved C15 2.01 mm to (164.0, 108.5)
- moved C14 2.01 mm to (167.5, 108.5)
Routing:
- net +5V: track 24.7 -> 22.7 mm
- net GND: track 48.7 -> 48.2 mm, vias 18 -> 19
Changed lines of the file:
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@@
 	(footprint "Capacitor_SMD:C_0805_2012Metric"
 		(layer "B.Cu")
-		(at 165.5 108.45 90)
+		(at 167.51 108.5 90)
 		(descr "Capacitor SMD 0805 (2012 Metric), square (rectangular) end terminal, IPC_7351 nominal, (Body size source: IPC-SM-782 page 76, https://www.pcb-3d.com/wordpress/wp-content/uploads/ipc-sm-782a_amendment_1_and_2.pdf, https://docs.google.com/spreadsheets/d/1BsfQQcO9C6DZCsRaXUlFlo91Tg2WpOkGARC1WS5S8t0/edit?usp=sharing), generated with kicad-footprint-generator")
 		(tags "capacitor")
@@
 		)
 		(property "Value" "10uF"
-			(at 0 -1.68 270)
+			(at -2.73 -0.81 180)
 			(layer "B.Fab")
 			(effects
@@
 	(footprint "Capacitor_SMD:C_0805_2012Metric"
 		(layer "B.Cu")
-		(at 162 108.49 90)
+		(at 164.01 108.54 90)
 		(descr "Capacitor SMD 0805 (2012 Metric), square (rectangular) end terminal, IPC_7351 nominal, (Body size source: IPC-SM-782 page 76, https://www.pcb-3d.com/wordpress/wp-content/uploads/ipc-sm-782a_amendment_1_and_2.pdf, https://docs.google.com/spreadsheets/d/1BsfQQcO9C6DZCsRaXUlFlo91Tg2WpOkGARC1WS5S8t0/edit?usp=sharing), generated with kicad-footprint-generator")
 		(tags "capacitor")
@@
 		)
 		(property "Value" "0.1uF"
-			(at 0 -1.68 270)
+			(at -2.67 -0.2 180)
 			(layer "B.Fab")
 			(effects
@@
 	)
 	(segment
-		(start 165.5 107.5)
-		(end 162.04 107.5)
+		(start 167.51 107.55)
+		(end 164.05 107.55)
 		(width 0.4)
 		(layer "B.Cu")
@@
 	)
 	(segment
+		(start 164.01 107.59)
+		(end 162.51 107.59)
+		(width 0.4)
+		(layer "B.Cu")
+		(net 4)
+	)
+	(segment
 		(start 123.81401 85.22401)
 		(end 123.87401 85.22401)
@@
 	)
 	(segment
-		(start 165.5 107.5)
-		(end 166.106 106.894)
-		(width 0.4)
-		(layer "B.Cu")
-		(net 4)
-	)
-	(segment
 		(start 123.87401 85.22401)
 		(end 124.688775 86.038775)
@@
 	)
 	(segment
-		(start 166.106 106.894)
-		(end 170.136 106.894)
-		(width 0.4)
+		(start 130.684747 79.121751)
+		(end 130.603249 79.121751)
+		(width 0.2)
 		(layer "B.Cu")
 		(net 4)
 	)
 	(segment
-		(start 130.684747 79.121751)
-		(end 130.603249 79.121751)
-		(width 0.2)
+		(start 170.16 106.87)
+		(end 168.19 106.87)
+		(width 0.4)
 		(layer "B.Cu")
 		(net 4)
@@
 	)
 	(segment
-		(start 162.04 107.5)
-		(end 162 107.54)
-		(width 0.2)
-		(layer "B.Cu")
-		(net 4)
-	)
-	(segment
 		(start 117.33953 77.31047)
 		(end 116.47 78.18)
@@
 	)
 	(segment
+		(start 168.19 106.87)
+		(end 167.51 107.55)
+		(width 0.4)
+		(layer "B.Cu")
+		(net 4)
+	)
+	(segment
 		(start 122.697024 78.950526)
 		(end 121.758775 79.888775)
@@
 	)
 	(via micro
+		(at 162.51 107.59)
+		(size 0.3)
+		(drill 0.1)
+		(layers "In2.Cu" "B.Cu")
+		(net 4)
+	)
+	(via micro
 		(at 128.78 106.76)
 		(size 0.3)
@@
 	)
 	(segment
+		(start 167.51 109.45)
+		(end 164.05 109.45)
+		(width 0.4)
+		(layer "B.Cu")
+		(net 6)
+	)
+	(segment
 		(start 132.887168 85.183312)
 		(end 132.883312 85.183312)
@@
 	)
 	(segment
-		(start 165.5 109.4)
-		(end 165.57 109.47)
-		(width 0.4)
-		(layer "B.Cu")
-		(net 6)
-	)
-	(segment
 		(start 100.17 92.13)
 		(end 100.18 92.12)
@@
 	)
 	(segment
-		(start 162.04 109.4)
-		(end 162 109.44)
-		(width 0.2)
-		(layer "B.Cu")
-		(net 6)
-	)
-	(segment
 		(start 134.225 79.975)
 		(end 133.525 79.275)
@@
 	)
 	(segment
-		(start 155.292606 120.154098)
-		(end 153.464512 118.326004)
+		(start 164.05 109.45)
+		(end 164.01 109.49)
 		(width 0.2)
 		(layer "B.Cu")
@@
 	)
 	(segment
-		(start 132.028249 77.778249)
-		(end 131.946751 77.778249)
+		(start 155.292606 120.154098)
+		(end 153.464512 118.326004)
 		(width 0.2)
 		(layer "B.Cu")
@@
 	)
 	(segment
-		(start 165.57 109.47)
-		(end 170.16 109.47)
-		(width 0.4)
+		(start 132.028249 77.778249)
+		(end 131.946751 77.778249)
+		(width 0.2)
 		(layer "B.Cu")
 		(net 6)
 	)
 	(segment
-		(start 165.5 109.4)
-		(end 162.04 109.4)
+		(start 170.16 109.47)
+		(end 167.53 109.47)
 		(width 0.4)
 		(layer "B.Cu")
@@
 		(net_name "")
 		(layer "B.Cu")
+		(name "GND")
 		(hatch edge 0.5)
 		(connect_pads
@@
 		(filled_areas_thickness no)
 		(keepout
-			(tracks allowed)
-			(vias allowed)
-			(pads allowed)
+			(tracks not_allowed)
+			(vias not_allowed)
+			(pads not_allowed)
 			(copperpour not_allowed)
 			(footprints allowed)
@@
 		(polygon
 			(pts
-				(xy 169.262077 104.18) (xy 162.741391 104.18) (xy 162.620825 112.077137) (xy 169.322532 112.039309)
+				(xy 125.26 79.71) (xy 124.24 78.66) (xy 123.86 78.79) (xy 122.94 79.96) (xy 122.75 80.15) (xy 123.81 81.33)
+				(xy 125.26 79.7)
 			)
 		)
@@
 		(filled_areas_thickness no)
 		(keepout
-			(tracks not_allowed)
-			(vias not_allowed)
-			(pads not_allowed)
+			(tracks allowed)
+			(vias allowed)
+			(pads allowed)
 			(copperpour not_allowed)
 			(footprints allowed)
@@
 		(polygon
 			(pts
-				(xy 125.26 79.71) (xy 124.24 78.66) (xy 123.86 78.79) (xy 122.94 79.96) (xy 122.75 80.15) (xy 123.81 81.33)
-				(xy 125.26 79.7)
+				(xy 133.77 84.54) (xy 133.21 84.5) (xy 132.87 84.86) (xy 133.21 85.2) (xy 133.21 85.17)
 			)
 		)
@@
 		(polygon
 			(pts
-				(xy 133.77 84.54) (xy 133.21 84.5) (xy 132.87 84.86) (xy 133.21 85.2) (xy 133.21 85.17)
+				(xy 149.76 118.27) (xy 147.37 115.89) (xy 145.52 117.75) (xy 147.9 120.03) (xy 149.76 118.25)
 			)
 		)
@@
 		(filled_areas_thickness no)
 		(keepout
-			(tracks allowed)
-			(vias allowed)
-			(pads allowed)
+			(tracks not_allowed)
+			(vias not_allowed)
+			(pads not_allowed)
 			(copperpour not_allowed)
 			(footprints allowed)
@@
 		(polygon
 			(pts
-				(xy 149.76 118.27) (xy 147.37 115.89) (xy 145.52 117.75) (xy 147.9 120.03) (xy 149.76 118.25)
+				(xy 131.74 83.38) (xy 131.93 83.17) (xy 128.57 80) (xy 128.18 80.4) (xy 129.03 81.2) (xy 128.17 82.58)
+				(xy 129.31 83.69) (xy 130.63 82.77) (xy 131.64 83.49) (xy 131.81 83.3)
 			)
 		)
@@
 		(filled_areas_thickness no)
 		(keepout
-			(tracks not_allowed)
-			(vias not_allowed)
-			(pads not_allowed)
+			(tracks allowed)
+			(vias allowed)
+			(pads allowed)
 			(copperpour not_allowed)
 			(footprints allowed)
@@
 		(polygon
 			(pts
-				(xy 131.74 83.38) (xy 131.93 83.17) (xy 128.57 80) (xy 128.18 80.4) (xy 129.03 81.2) (xy 128.17 82.58)
-				(xy 129.31 83.69) (xy 130.63 82.77) (xy 131.64 83.49) (xy 131.81 83.3)
+				(xy 135.9 92.81) (xy 131.43 88.53) (xy 128.36 91.72) (xy 132.638815 96.160966)
 			)
 		)
@@
 		(polygon
 			(pts
-				(xy 135.9 92.81) (xy 131.43 88.53) (xy 128.36 91.72) (xy 132.638815 96.160966)
+				(xy 146.23 117.01) (xy 143.0725 120.2425) (xy 140.950937 120.258931) (xy 127.957644 107.362802)
+				(xy 127.975225 106.095411) (xy 131.130478 103.1329) (xy 132.312899 103.150097)
 			)
 		)
@@
 		(polygon
 			(pts
-				(xy 146.23 117.01) (xy 143.0725 120.2425) (xy 140.950937 120.258931) (xy 127.957644 107.362802)
-				(xy 127.975225 106.095411) (xy 131.130478 103.1329) (xy 132.312899 103.150097)
+				(xy 134.85 87.85) (xy 134.44 87.47) (xy 131.01 87.25) (xy 130.75 87.48) (xy 133.66 90.38) (xy 134.12 90.04)
+				(xy 133.7 89.5) (xy 133.82 89.06) (xy 134.91 87.93) (xy 134.81 87.82)
 			)
 		)
@@
 		(net_name "")
 		(layer "B.Cu")
-		(name "GND")
 		(hatch edge 0.5)
 		(connect_pads
@@
 		(placement
 			(enabled no)
-			(sheetname "/Power/")
+			(sheetname "")
 		)
 		(fill
@@
 		(polygon
 			(pts
-				(xy 134.85 87.85) (xy 134.44 87.47) (xy 131.01 87.25) (xy 130.75 87.48) (xy 133.66 90.38) (xy 134.12 90.04)
-				(xy 133.7 89.5) (xy 133.82 89.06) (xy 134.91 87.93) (xy 134.81 87.82)
+				(xy 170.85 106.62) (xy 170.85 109.77) (xy 171.805 109.76) (xy 171.805 106.62)
 			)
 		)
@@
 			)
 		)
+	)
+	(zone
+		(net 0)
+		(net_name "")
+		(layer "B.Cu")
+		(hatch edge 0.5)
+		(connect_pads
+			(clearance 0)
+		)
+		(min_thickness 0.25)
+		(filled_areas_thickness no)
+		(keepout
+			(tracks allowed)
+			(vias allowed)
+			(pads allowed)
+			(copperpour not_allowed)
+			(footprints allowed)
+		)
+		(placement
+			(enabled no)
+			(sheetname "")
+		)
+		(fill
+			(thermal_gap 0.5)
+			(thermal_bridge_width 0.5)
+		)
+		(polygon
+			(pts
+				(xy 169.35 105.67) (xy 169.35 111.55) (xy 161.4 111.6) (xy 161.37 105.66)
+			)
+		)
