File: hardware/muon_pcb/muon_pcb.kicad_sch (KiCad schematic)
At the start: 0 parts

Commit message: work in progress on updating schematic and layout
Other:
- note added: "Communications"
- note removed: "Cosmic Bridge"
