File: hardware/Cygnet Skywalker v1/Cygnet Skywalker v1.kicad_pcb (KiCad board)
At the start: 4 copper layers, 88 x 94.5 mm, 146 parts, among them J1 USB_B_Micro, J10 BM04B-SRSS-TB(LF)(SN), J11 Conn_Coaxial, J12 Conn_01x02, J2 Hirose DF11 02x06, J3 SWD Port, J4 Hirose DF11 02x06, J5 BM04B-SRSS-TB(LF)(SN), J6 BM04B-SRSS-TB(LF)(SN), J7 BM04B-SRSS-TB(LF)(SN), J8 BM04B-SRSS-TB(LF)(SN), J9 BM04B-SRSS-TB(LF)(SN), SW1 SW_Push, SW2 SW_Push, U1 W25Q128JVS, U10 INA260, U11 RM-VT01-A Readout Module, U12 RM-VT01-A Readout Module, U13 Skytraq Orion B16 GPS, U14 TPS22992, U15 TLV1704, U2 TLV76733DGNR, U3 TPS62142, U4 RP2350_60QFN_C42411118, U5 TLV61048, U6 INA260, U7 INA260, U8 INA260, U9 TMP117xxDRV, Y1 ABM8-272-T3

Commit message: remove layout
yipeee
Parts:
- removed C1, C2: 15p, Capacitor_SMD:C_0402_1005Metric
- removed C10, C11, C5, C6: 4.7u, Capacitor_SMD:C_0402_1005Metric
- removed C12: 3.3nF, Capacitor_SMD:C_0603_1608Metric
- removed C13, C15, C17, C18, C19, C20, C21, C23, C29, C30, C31, C33, C34, C37, C4, C8: 100n, Capacitor_SMD:C_0402_1005Metric
- removed C14: 22u, Capacitor_SMD:C_1206_3216Metric
- removed C16, C3, C7: 1u, Capacitor_SMD:C_0603_1608Metric
- removed C22, C32, C35: 10u, Capacitor_SMD:C_1206_3216Metric
- removed C24, C25, C26, C27, C28, C36, C9: 10u, Capacitor_SMD:C_0805_2012Metric
- removed C38: 2.7n, Capacitor_SMD:C_0603_1608Metric
- removed C39, C40, C41, C42, C43: 10uF, Capacitor_SMD:C_0603_1608Metric
- removed D1, D7, D8: RED, LED_SMD:LED_0603_1608Metric
- removed D10, D9: YELLOW, LED_SMD:LED_0603_1608Metric
- removed D11, D2: B120AF-13, Skywalkerfeet:B120AF-13
- removed D12, D3: GREEN, LED_SMD:LED_0603_1608Metric
- removed D13: 1N4151WS, Diode_SMD:D_SOD-323
- removed D4: BLUE, LED_SMD:LED_0603_1608Metric
- removed D5: WHITE, LED_SMD:LED_0603_1608Metric
- removed D6: NSR0320, Diode_SMD:D_SOD-323F
- removed G*** (x2): LOGO, LOGO
- removed G***: LOGO, 1my_footprints:cadence_cygnet_logo_placeholder
- removed J1: USB_B_Micro, Skywalkerfeet:MICRO-USB-SMD_10118194-0001LF
- removed J10, J5, J6, J7, J8, J9: BM04B-SRSS-TB(LF)(SN), Skywalkerfeet:BM04B-SRSS-TB(LF)(SN)
- removed J11: Conn_Coaxial, Skywalkerfeet:SMA-TH_132134
- removed J12: Conn_01x02, Connector_PinHeader_2.54mm:PinHeader_1x02_P2.54mm_Vertical
- removed J2, J4: Hirose DF11 02x06, Connector_Hirose:Hirose_DF11-12DP-2DSA_2x06_P2.00mm_Vertical
- removed J3: SWD Port, Connector_PinHeader_1.27mm:PinHeader_2x02_P1.27mm_Vertical
- removed JP1: SolderJumper_2_Open, Jumper:SolderJumper-2_P1.3mm_Open_RoundedPad1.0x1.5mm
- removed L1: 3.3u, Skywalkerfeet:L_pol_2016
- removed L2: 2.2uH, Inductor_SMD:L_Coilcraft_XxL4020
- removed L3: 4.7uH, Skywalkerfeet:SWPA5040S4R7NT
- removed R1, R13, R5: 10k, Resistor_SMD:R_0402_1005Metric
- removed R10: 33, Resistor_SMD:R_0402_1005Metric
- removed R11: 10k, Capacitor_SMD:C_0402_1005Metric
- removed R12, R14, R15, R16, R25, R26, R27, R31, R32: 10k, Resistor_SMD:R_0603_1608Metric
- removed R17, R18: 27, Resistor_SMD:R_0402_1005Metric
- removed R19, R20, R23, R24, R41: 4.7k, Resistor_SMD:R_0402_1005Metric
- removed R2, R7, R9: 1k, Resistor_SMD:R_0402_1005Metric
- removed R21: 1.5M, Resistor_SMD:R_0603_1608Metric
- removed R22: 107k, Resistor_SMD:R_0603_1608Metric
- removed R28, R29, R30: 3.0k, Resistor_SMD:R_0603_1608Metric
- removed R3: 220, Resistor_SMD:R_0603_1608Metric
- removed R33, R35: 1k, Resistor_SMD:R_0603_1608Metric
- removed R34, R36, R37, R38, R40: 100k, Resistor_SMD:R_0603_1608Metric
- removed R39: 4.7M, Resistor_SMD:R_0603_1608Metric
- removed R4: 470, Resistor_SMD:R_0603_1608Metric
- removed R6: 1.47k, Resistor_SMD:R_0603_1608Metric
- removed R8: 330, Resistor_SMD:R_0603_1608Metric
- removed SW1, SW2: SW_Push, Skywalkerfeet:KEY-SMD_KMR2XXGXXX
- removed TP1: 3.3V Testpoint, Skywalkerfeet:Keystone5001_Testpoint
- removed TP10, TP8, TP9: GND, Skywalkerfeet:Keystone5001_Testpoint
- removed TP2: Module1 Vo, Skywalkerfeet:Keystone5001_Testpoint
- removed TP3: 5V Testpoint, Skywalkerfeet:Keystone5001_Testpoint
- removed TP4: Module2 Vo, Skywalkerfeet:Keystone5001_Testpoint
- removed TP5: 12V Testpoint, Skywalkerfeet:Keystone5001_Testpoint
- removed TP6: GPS 1PPS, Skywalkerfeet:Keystone5001_Testpoint
- removed TP7: 7V Testpoint, Skywalkerfeet:Keystone5001_Testpoint
- removed U1: W25Q128JVS, Package_SO:SOIC-8_5.3x5.3mm_P1.27mm
- removed U10, U6, U7, U8: INA260, Package_SO:TSSOP-16_4.4x5mm_P0.65mm
- removed U11, U12: RM-VT01-A Readout Module, Skywalkerfeet:RM-VT01-A
- removed U13: Skytraq Orion B16 GPS, Skywalkerfeet:Skytraq Orion B16 GPS
- removed U14: TPS22992, Skywalkerfeet:TPS22992
- removed U15: TLV1704, Package_SO:TSSOP-14_4.4x5mm_P0.65mm
- removed U2: TLV76733DGNR, Skywalkerfeet:TLV76733DGNR
- removed U3: TPS62142, Package_DFN_QFN:VQFN-16-1EP_3x3mm_P0.5mm_EP1.68x1.68mm_ThermalVias
- removed U4: RP2350_60QFN_C42411118, Skywalkerfeet:RP2350-QFN-60-1EP_7x7_P0.4mm_EP3.4x3.4mm_ThermalVias
- removed U5: TLV61048, Package_TO_SOT_SMD:SOT-23-6
- removed U9: TMP117xxDRV, Package_SON:WSON-6-1EP_2x2mm_P0.65mm_EP1x1.6mm
- removed Y1: ABM8-272-T3, Skywalkerfeet:ABM8-272-T3
Routing:
- net SCL1: track 135.6 -> 0.00 mm, vias 6 -> 0
- net +12V: track 134.1 -> 0.00 mm
- net SDA1: track 133.3 -> 0.00 mm, vias 9 -> 0
- net PAYLOAD_BATT_OUT: track 114.0 -> 0.00 mm, vias 2 -> 0
- net +3.3V: track 108.4 -> 0.00 mm, vias 62 -> 0
- net PET DOG: track 90.8 -> 0.00 mm, vias 2 -> 0
- net DOG Bite: track 86.3 -> 0.00 mm, vias 3 -> 0
- net Module1 R2 CTRL: track 78.2 -> 0.00 mm, vias 2 -> 0
- net Module1 Enable CTRL: track 75.3 -> 0.00 mm, vias 2 -> 0
- net Module1 R1 CTRL: track 70.3 -> 0.00 mm, vias 2 -> 0
- net GPS 1PPS: track 65.8 -> 0.00 mm, vias 1 -> 0
- net UART0 Rx: track 56.1 -> 0.00 mm, vias 3 -> 0
- net Module2 R1 CTRL: track 55.6 -> 0.00 mm, vias 2 -> 0
- net Module2 Enable CTRL: track 55.2 -> 0.00 mm, vias 2 -> 0
- net Module2 R2 CTRL: track 54.8 -> 0.00 mm, vias 2 -> 0
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- removed copper zone on F.Cu, net (none)
- removed copper zone on F.Cu, net +1V1
- removed copper zone on F.Cu, net +3.3V
- removed copper zone on In2.Cu, net +3.3V
- removed copper zone on B.Cu, net GND
- removed copper zone on F.Cu, net GND
- removed copper zone on In1.Cu, net GND
Other:
- board text removed: "12V"
- board text removed: "3.3V"
- board text removed: "5V"
- board text removed: "7V"
- board text removed: "CYGNET RADFET Payload Board by William Hsu & Max Gross With Michael Pham's Stamp of Approval!"
- board text removed: "Cygnet Skywalker v1"
- board text removed: "Flash RSET"
- board text removed: "GND"
- board text removed: "GPIO Breakout"
- board text removed: "GPS 1PPS"
- board text removed: "GPS Coaxial"
- board text removed: "I2C0 Debug"
- board text removed: "I2C1 Debug"
- board text removed: "MCU RSET"
- board text removed: "Made with JLCPCB :)"
- board text removed: "Module 1 Vout"
- board text removed: "Module 2 Vout"
- board text removed: "PROVES FC"
- board text removed: "RADFET Module 1"
- board text removed: "RADFET Module 2"
- board text removed: "SWDs & RSet Debug"
- board text removed: "Solder to enable Watchdog ---->"
- board text removed: "Thank you Bouni for making the BOM making process less painful!"
- board text removed: "UART0 Debug"
- board text removed: "UART1 Debug"
- board text removed: "USB Debug"
- board text removed: "{dblquote}You were the chosen one! It was said that you would destroy the Sith, not join them! Bring balance to the Force, not leave it in darkness!{dblquote}"

Commit message: layouts
Parts:
- added C1: 15p, Capacitor_SMD:C_0402_1005Metric, F.Cu at (329.5, 130.8)
- added C10: 4.7u, Capacitor_SMD:C_0402_1005Metric, F.Cu at (332.4, 130.8)
- added C11: 4.7u, Capacitor_SMD:C_0402_1005Metric, F.Cu at (332.4, 132.7)
- added C12: 3.3nF, Capacitor_SMD:C_0603_1608Metric, F.Cu at (338.5, 122.0)
- added C13: 100n, Capacitor_SMD:C_0402_1005Metric, F.Cu at (332.4, 134.7)
- added C14: 22u, Capacitor_SMD:C_1206_3216Metric, F.Cu at (323.3, 150.4)
- added C15: 100n, Capacitor_SMD:C_0402_1005Metric, F.Cu at (332.4, 136.7)
- added C16: 1u, Capacitor_SMD:C_0603_1608Metric, F.Cu at (338.5, 124.5)
- added C17: 100n, Capacitor_SMD:C_0402_1005Metric, F.Cu at (332.4, 138.6)
- added C18: 100n, Capacitor_SMD:C_0402_1005Metric, F.Cu at (332.4, 140.6)
- added C19: 100n, Capacitor_SMD:C_0402_1005Metric, F.Cu at (335.2, 130.8)
- added C2: 15p, Capacitor_SMD:C_0402_1005Metric, F.Cu at (329.5, 132.7)
- added C20: 100n, Capacitor_SMD:C_0402_1005Metric, F.Cu at (335.2, 132.7)
- added C21: 100n, Capacitor_SMD:C_0402_1005Metric, F.Cu at (335.2, 134.7)
- added C22: 10u, Capacitor_SMD:C_1206_3216Metric, F.Cu at (323.3, 153.8)
- added C23: 100n, Capacitor_SMD:C_0402_1005Metric, F.Cu at (335.2, 136.7)
- added C24: 10u, Capacitor_SMD:C_0805_2012Metric, F.Cu at (343.0, 144.2)
- added C25: 10u, Capacitor_SMD:C_0805_2012Metric, F.Cu at (343.0, 147.2)
- added C26: 10u, Capacitor_SMD:C_0805_2012Metric, F.Cu at (343.0, 150.3)
- added C27: 10u, Capacitor_SMD:C_0805_2012Metric, F.Cu at (343.0, 153.3)
- added C28: 10u, Capacitor_SMD:C_0805_2012Metric, F.Cu at (343.0, 156.3)
- added C29: 100n, Capacitor_SMD:C_0402_1005Metric, F.Cu at (328.9, 97.6)
- added C3: 1u, Capacitor_SMD:C_0603_1608Metric, F.Cu at (338.5, 116.9)
- added C30: 100n, Capacitor_SMD:C_0402_1005Metric, F.Cu at (328.9, 99.5)
- added C31: 100n, Capacitor_SMD:C_0402_1005Metric, F.Cu at (328.9, 101.5)
- added C32: 10u, Capacitor_SMD:C_1206_3216Metric, F.Cu at (333.2, 106.8)
- added C33: 100n, Capacitor_SMD:C_0402_1005Metric, F.Cu at (328.9, 103.5)
- added C34: 100n, Capacitor_SMD:C_0402_1005Metric, F.Cu at (328.9, 105.4)
- added C35: 10u, Capacitor_SMD:C_1206_3216Metric, F.Cu at (333.2, 110.2)
- added C36: 10u, Capacitor_SMD:C_0805_2012Metric, F.Cu at (341.2, 98.1)
- added C37: 100n, Capacitor_SMD:C_0402_1005Metric, F.Cu at (328.9, 107.4)
- added C38: 2.7n, Capacitor_SMD:C_0603_1608Metric, F.Cu at (340.9, 100.8)
- added C39: 10uF, Capacitor_SMD:C_0603_1608Metric, F.Cu at (361.5, 116.9)
- added C4: 100n, Capacitor_SMD:C_0402_1005Metric, F.Cu at (329.5, 134.7)
- added C40: 10uF, Capacitor_SMD:C_0603_1608Metric, F.Cu at (361.5, 119.4)
- added C41: 10uF, Capacitor_SMD:C_0603_1608Metric, F.Cu at (361.5, 122.0)
- added C42: 10uF, Capacitor_SMD:C_0603_1608Metric, F.Cu at (361.5, 124.5)
- added C43: 10uF, Capacitor_SMD:C_0603_1608Metric, F.Cu at (361.5, 127.0)
- added C5: 4.7u, Capacitor_SMD:C_0402_1005Metric, F.Cu at (329.5, 136.7)
- added C6: 4.7u, Capacitor_SMD:C_0402_1005Metric, F.Cu at (329.5, 138.6)
- added C7: 1u, Capacitor_SMD:C_0603_1608Metric, F.Cu at (338.5, 119.4)
- added C8: 100n, Capacitor_SMD:C_0402_1005Metric, F.Cu at (329.5, 140.6)
- added C9: 10u, Capacitor_SMD:C_0805_2012Metric, F.Cu at (343.0, 141.2)
- added D1: RED, LED_SMD:LED_0603_1608Metric, F.Cu at (338.7, 141.0)
- added D10: YELLOW, LED_SMD:LED_0603_1608Metric, F.Cu at (338.7, 159.2)
- added D11: B120AF-13, Skywalkerfeet:B120AF-13, F.Cu at (332.0, 148.1)
- added D12: GREEN, LED_SMD:LED_0603_1608Metric, F.Cu at (378.1, 117.0)
- added D13: 1N4151WS, Diode_SMD:D_SOD-323, F.Cu at (378.0, 131.0)
- added D2: B120AF-13, Skywalkerfeet:B120AF-13, F.Cu at (332.0, 143.8)
- added D3: GREEN, LED_SMD:LED_0603_1608Metric, F.Cu at (338.7, 143.6)
- added D4: BLUE, LED_SMD:LED_0603_1608Metric, F.Cu at (338.7, 146.2)
- added D5: WHITE, LED_SMD:LED_0603_1608Metric, F.Cu at (338.7, 148.8)
- added D6: NSR0320, Diode_SMD:D_SOD-323F, F.Cu at (314.9, 158.4)
- added D7: RED, LED_SMD:LED_0603_1608Metric, F.Cu at (338.7, 151.4)
- added D8: RED, LED_SMD:LED_0603_1608Metric, F.Cu at (338.7, 154.0)
- added D9: YELLOW, LED_SMD:LED_0603_1608Metric, F.Cu at (338.7, 156.6)
- added J1: USB_B_Micro, Skywalkerfeet:MICRO-USB-SMD_10118194-0001LF, F.Cu at (349.8, 149.2)
- added J10: BM04B-SRSS-TB(LF)(SN), Skywalkerfeet:BM04B-SRSS-TB(LF)(SN), F.Cu at (316.6, 144.3)
- added J11: Conn_Coaxial, Skywalkerfeet:SMA-TH_132134, F.Cu at (334.6, 100.9)
- added J12: Conn_01x02, Connector_PinHeader_2.54mm:PinHeader_1x02_P2.54mm_Vertical, F.Cu at (373.8, 118.0)
- added J2: Hirose DF11 02x06, Connector_Hirose:Hirose_DF11-12DP-2DSA_2x06_P2.00mm_Vertical, F.Cu at (323.5, 118.2)
- added J3: SWD Port, Connector_PinHeader_1.27mm:PinHeader_2x02_P1.27mm_Vertical, F.Cu at (322.6, 157.1)
- added J4: Hirose DF11 02x06, Connector_Hirose:Hirose_DF11-12DP-2DSA_2x06_P2.00mm_Vertical, F.Cu at (323.5, 125.2)
- added J5: BM04B-SRSS-TB(LF)(SN), Skywalkerfeet:BM04B-SRSS-TB(LF)(SN), F.Cu at (316.6, 118.3)
- added J6: BM04B-SRSS-TB(LF)(SN), Skywalkerfeet:BM04B-SRSS-TB(LF)(SN), F.Cu at (316.6, 123.5)
- added J7: BM04B-SRSS-TB(LF)(SN), Skywalkerfeet:BM04B-SRSS-TB(LF)(SN), F.Cu at (316.6, 128.7)
- added J8: BM04B-SRSS-TB(LF)(SN), Skywalkerfeet:BM04B-SRSS-TB(LF)(SN), F.Cu at (316.6, 133.9)
- added J9: BM04B-SRSS-TB(LF)(SN), Skywalkerfeet:BM04B-SRSS-TB(LF)(SN), F.Cu at (316.6, 139.1)
- added JP1: SolderJumper_2_Open, Jumper:SolderJumper-2_P1.3mm_Open_RoundedPad1.0x1.5mm, F.Cu at (373.7, 131.3)
- added L1: 3.3u, Skywalkerfeet:L_pol_2016, F.Cu at (354.9, 117.7)
- added L2: 2.2uH, Inductor_SMD:L_Coilcraft_XxL4020, F.Cu at (351.4, 125.5)
- added L3: 4.7uH, Skywalkerfeet:SWPA5040S4R7NT, F.Cu at (348.7, 156.9)
- added R1: 10k, Resistor_SMD:R_0402_1005Metric, F.Cu at (338.1, 130.8)
- added R10: 33, Resistor_SMD:R_0402_1005Metric, F.Cu at (341.0, 130.8)
- added R11: 10k, Capacitor_SMD:C_0402_1005Metric, F.Cu at (335.2, 138.6)
- added R12: 10k, Resistor_SMD:R_0603_1608Metric, F.Cu at (342.6, 124.5)
- added R13: 10k, Resistor_SMD:R_0402_1005Metric, F.Cu at (341.0, 132.8)
- added R14: 10k, Resistor_SMD:R_0603_1608Metric, F.Cu at (342.6, 127.0)
- added R15: 10k, Resistor_SMD:R_0603_1608Metric, F.Cu at (346.6, 116.9)
- added R16: 10k, Resistor_SMD:R_0603_1608Metric, F.Cu at (346.6, 119.4)
- added R17: 27, Resistor_SMD:R_0402_1005Metric, F.Cu at (341.0, 134.8)
- added R18: 27, Resistor_SMD:R_0402_1005Metric, F.Cu at (341.0, 136.7)
- added R19: 4.7k, Resistor_SMD:R_0402_1005Metric, F.Cu at (341.0, 138.7)
- added R2: 1k, Resistor_SMD:R_0402_1005Metric, F.Cu at (338.1, 132.8)
- added R20: 4.7k, Resistor_SMD:R_0402_1005Metric, F.Cu at (344.0, 130.8)
- added R21: 1.5M, Resistor_SMD:R_0603_1608Metric, F.Cu at (346.6, 122.0)
- added R22: 107k, Resistor_SMD:R_0603_1608Metric, F.Cu at (346.6, 124.5)
- added R23: 4.7k, Resistor_SMD:R_0402_1005Metric, F.Cu at (344.0, 132.8)
- added R24: 4.7k, Resistor_SMD:R_0402_1005Metric, F.Cu at (344.0, 134.8)
- added R25: 10k, Resistor_SMD:R_0603_1608Metric, F.Cu at (361.5, 129.5)
- added R26: 10k, Resistor_SMD:R_0603_1608Metric, F.Cu at (361.5, 132.0)
- added R27: 10k, Resistor_SMD:R_0603_1608Metric, F.Cu at (365.5, 116.9)
- added R28: 3.0k, Resistor_SMD:R_0603_1608Metric, F.Cu at (365.5, 119.4)
- added R29: 3.0k, Resistor_SMD:R_0603_1608Metric, F.Cu at (365.5, 122.0)
- added R3: 220, Resistor_SMD:R_0603_1608Metric, F.Cu at (338.5, 127.0)
- added R30: 3.0k, Resistor_SMD:R_0603_1608Metric, F.Cu at (365.5, 124.5)
- added R31: 10k, Resistor_SMD:R_0603_1608Metric, F.Cu at (365.5, 127.0)
- added R32: 10k, Resistor_SMD:R_0603_1608Metric, F.Cu at (365.5, 129.5)
- added R33: 1k, Resistor_SMD:R_0603_1608Metric, F.Cu at (365.5, 132.0)
- added R34: 100k, Resistor_SMD:R_0603_1608Metric, F.Cu at (369.5, 116.9)
- added R35: 1k, Resistor_SMD:R_0603_1608Metric, F.Cu at (369.5, 119.4)
- added R36: 100k, Resistor_SMD:R_0603_1608Metric, F.Cu at (369.5, 122.0)
- added R37: 100k, Resistor_SMD:R_0603_1608Metric, F.Cu at (369.5, 124.5)
- added R38: 100k, Resistor_SMD:R_0603_1608Metric, F.Cu at (369.5, 127.0)
- added R39: 4.7M, Resistor_SMD:R_0603_1608Metric, F.Cu at (369.5, 129.5)
- added R4: 470, Resistor_SMD:R_0603_1608Metric, F.Cu at (342.6, 116.9)
- added R40: 100k, Resistor_SMD:R_0603_1608Metric, F.Cu at (369.5, 132.0)
- added R41: 4.7k, Resistor_SMD:R_0402_1005Metric, F.Cu at (340.4, 110.2)
- added R5: 10k, Resistor_SMD:R_0402_1005Metric, F.Cu at (338.1, 134.8)
- added R6: 1.47k, Resistor_SMD:R_0603_1608Metric, F.Cu at (342.6, 119.4)
- added R7: 1k, Resistor_SMD:R_0402_1005Metric, F.Cu at (338.1, 136.7)
- added R8: 330, Resistor_SMD:R_0603_1608Metric, F.Cu at (342.6, 122.0)
- added R9: 1k, Resistor_SMD:R_0402_1005Metric, F.Cu at (338.1, 138.7)
- added SW1: SW_Push, Skywalkerfeet:KEY-SMD_KMR2XXGXXX, F.Cu at (331.4, 152.3)
- added SW2: SW_Push, Skywalkerfeet:KEY-SMD_KMR2XXGXXX, F.Cu at (331.4, 156.7)
- added TP1: 3.3V Testpoint, Skywalkerfeet:Keystone5001_Testpoint, F.Cu at (322.4, 131.7)
- added TP10: GND, Skywalkerfeet:Keystone5001_Testpoint, F.Cu at (326.2, 146.8)
- added TP2: Module1 Vo, Skywalkerfeet:Keystone5001_Testpoint, F.Cu at (322.4, 135.5)
- added TP3: 5V Testpoint, Skywalkerfeet:Keystone5001_Testpoint, F.Cu at (322.4, 139.2)
- added TP4: Module2 Vo, Skywalkerfeet:Keystone5001_Testpoint, F.Cu at (322.4, 143.0)
- added TP5: 12V Testpoint, Skywalkerfeet:Keystone5001_Testpoint, F.Cu at (322.4, 146.8)
- added TP6: GPS 1PPS, Skywalkerfeet:Keystone5001_Testpoint, F.Cu at (326.2, 131.7)
- added TP7: 7V Testpoint, Skywalkerfeet:Keystone5001_Testpoint, F.Cu at (326.2, 135.5)
- added TP8: GND, Skywalkerfeet:Keystone5001_Testpoint, F.Cu at (326.2, 139.2)
- added TP9: GND, Skywalkerfeet:Keystone5001_Testpoint, F.Cu at (326.2, 143.0)
- added U1: W25Q128JVS, Package_SO:SOIC-8_5.3x5.3mm_P1.27mm, F.Cu at (350.4, 143.3)
- added U10: INA260, Package_SO:TSSOP-16_4.4x5mm_P0.65mm, F.Cu at (354.8, 91.8)
- added U11: RM-VT01-A Readout Module, Skywalkerfeet:RM-VT01-A, F.Cu at (322.0, 69.5)
- added U12: RM-VT01-A Readout Module, Skywalkerfeet:RM-VT01-A, F.Cu at (340.7, 69.5)
- added U13: Skytraq Orion B16 GPS, Skywalkerfeet:Skytraq Orion B16 GPS, F.Cu at (320.1, 104.1)
- added U14: TPS22992, Skywalkerfeet:TPS22992, F.Cu at (341.2, 103.9)
- added U15: TLV1704, Package_SO:TSSOP-14_4.4x5mm_P0.65mm, F.Cu at (375.9, 126.3)
- added U2: TLV76733DGNR, Skywalkerfeet:TLV76733DGNR, F.Cu at (351.0, 119.2)
- added U3: TPS62142, Package_DFN_QFN:VQFN-16-1EP_3x3mm_P0.5mm_EP1.68x1.68mm_ThermalVias, F.Cu at (315.7, 149.5)
- added U4: RP2350_60QFN_C42411118, Skywalkerfeet:RP2350-QFN-60-1EP_7x7_P0.4mm_EP3.4x3.4mm_ThermalVias, F.Cu at (350.1, 134.4)
- added U5: TLV61048, Package_TO_SOT_SMD:SOT-23-6, F.Cu at (354.9, 156.2)
- added U6: INA260, Package_SO:TSSOP-16_4.4x5mm_P0.65mm, F.Cu at (354.8, 72.0)
- added U7: INA260, Package_SO:TSSOP-16_4.4x5mm_P0.65mm, F.Cu at (354.8, 78.6)
- added U8: INA260, Package_SO:TSSOP-16_4.4x5mm_P0.65mm, F.Cu at (354.8, 85.2)
- added U9: TMP117xxDRV, Package_SON:WSON-6-1EP_2x2mm_P0.65mm_EP1x1.6mm, F.Cu at (340.8, 107.4)
- added Y1: ABM8-272-T3, Skywalkerfeet:ABM8-272-T3, F.Cu at (315.5, 154.4)

Commit message: moved
rad team
Parts:
- moved D13 9.29 mm to (386.9, 133.6)
Changed lines of the file:
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@@
 	(footprint "Diode_SMD:D_SOD-323"
 		(layer "F.Cu")
-		(at 378 131)
+		(at 386.925 133.575)
 		(descr "SOD-323")
 		(tags "SOD-323")

Commit message: william
Parts:
- moved U13 74.9 mm to (248.3, 82.8)
Changed lines of the file:
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@@
 	(footprint "Skywalkerfeet:Skytraq Orion B16 GPS"
 		(layer "F.Cu")
-		(at 320.09125 104.075)
+		(at 248.275 82.825)
 		(property "Reference" "U13"
 			(at 0 -11.95 0)
