File: hardware/Radfet_breakout/Radfet_breakout.kicad_sch (KiCad schematic)
At the start: 0 parts

Commit message: pushing
pushing
Parts:
- added C1: 10u, symbol Device:C
- added J1: Conn_Coaxial_Small, symbol Connector:Conn_Coaxial_Small
- added J2: Conn_02x06_Counter_Clockwise, symbol Connector_Generic:Conn_02x06_Counter_Clockwise
- added U1: ~, symbol RadfETS:RadFETS
- added U2, U3: ATSAMV70N20B-AAB, TQFP100_14x14MC_MCH, symbol ATSAMV70N20:ATSAMV70N20B-AAB
Connections:
- new net +12V: C1.1, J2.1 (Pin_1), U1.1 (Vdd)
- new net EN: J2.3 (Pin_3), U1.5 (CTRL_EN)
- new net GND: C1.2, J1.2 (Ext), J2.5 (Pin_5), U1.2 (GND), U1.3 (GND), U2.10 (GND), U2.29 (GND), U2.3 (GND), U2.67 (GND), U2.7 (GND), U2.8 (GND)
- new net R1: J2.4 (Pin_4), U1.6 (CTRL_R1)
- new net R2: J2.2 (Pin_2), U1.4 (CTRL_R2)
- new net RadFET_Vo: J1.1 (In), U1.9 (RADFET_OUT)
- no-connect marks 0 -> 7
