File: hardware/i.MX8X Flight Computer Carrier Board/CADENCE i.MX8X Carrier Board rev1/imx8xsom.kicad_sch (KiCad schematic)
At the start: 110 parts, among them CN1 DF11-16DP-2DSA(08), CN2 DF11-16DP-2DSA(08), J1 Micro_SD_Card_Det1, J12 Conn_01x02, J2 USB_A, J3 Conn_Coaxial, J4 Conn_02x26_Odd_Even, J7 Conn_02x06_Odd_Even, J9 Conn_02x26_Odd_Even, SW1 SW_DIP_x04, U1 INA219AxDCN, U10 MR20H40, U11 LSM6DSO, U12 LIS2MDL, U14 MR20H40, U15 TLV1704, U2 INA219AxDCN, U20 ZDSD04GLGEAG, U24 TMP112xxDRL, U29 USBLC6-2SC6, U3 P82B715DR, U30 USBLC6-2SC6, U31 MAX3485, U32 P82B715DR, U4 P82B715DR, U6 Skytraq Orion B16 GPS, U7 AMS1117-3.3, U8 AMS1117-3.3, U9 RV-3028-C7

Commit message: updated to do list & labels
Other:
- note added: "I2C List: I2C0: onboard RTC, IMU sensors, Temperature Sensors I2C1: Power Monitors I2C2: electrical power system management board I2c3 & I2C4: payload board i2c4: adcs connection likely (must further research cubespace adcs interface control document and connections. also adcs is still uncertain)"
- note added: "I2C2 (Connection to EPS Board)"
- note added: "Not Sure if this is how rs422 is implemented or if it works this way. Must look into deeply first"
- note added: "TO DO: - reorganize & fully implement board to board connections (SATNOGS should only need i2c now but double check; payload needs few i2c bus and rs422 if possible;adcs connection needs to be implemented) - double check octal spi nor flash memory implementation (very briefly skimmed datasheet) - add heater and antenna trigger connection/connector (need to talk with thermals & power about interfa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"
- note added: "VBATT-->Regulator_Output-->3.3V"
- note added: "assign pin for output (likely to load switch to onboard power regulators/power load switch that allows for power cycling)"
- note added: "prob gonna nuke eeprom (nominally more likely to be affected by radiation) keeping for now in case mind changes"
- note added: "rs422 prob doesnt work this way. look into implementation and if we can use uart to rs422 or if we need dedicated ftdi chip or something"
- note removed: "I2C List: I2C0: RTC, IMU sensors, Temperature Sensors I2C1: Power Monitors"
- note removed: "I2C2 (Connection to Payload Board)"
- note removed: "TO DO: - assign i2c addresses to power monitors - reorganize board to board connections - double check memory implementations (ospi left now) - add heater and antenna trigger - add more watchdogs (for power, processor, satnogs) -assign watchdog input/output pins -add rs422 transceiver to payload connection"
- note removed: "assign pin for output"
- note removed: "gonna nuke eeprom (nominally more likely to be affected by radiation) keeping for now in case mind changes"
Changed lines of the file:
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@@
 		)
 	)
-	(text "I2C2 (Connection to Payload Board)"
+	(text "I2C2 (Connection to EPS Board)"
 		(exclude_from_sim no)
 		(at 259.08 109.22 0)
@@
 		)
 	)
+	(text "Payload Board Connection"
+		(exclude_from_sim no)
+		(at 552.196 539.496 0)
+		(effects
+			(font
+				(size 3.81 3.81)
+				(thickness 0.762)
+				(bold yes)
+			)
+		)
+	)
 	(text "connect to gpio on imx (1pps) maybe also add bootsel?"
 		(exclude_from_sim no)
@@
 		)
 	)
-	(text "I2C List:\nI2C0: RTC, IMU sensors, Temperature Sensors\nI2C1: Power Monitors\n"
+	(text "I2C List:\nI2C0: onboard RTC, IMU sensors, Temperature Sensors\nI2C1: Power Monitors\nI2C2: electrical power system management board\nI2c3 & I2C4: payload board\ni2c4: adcs connection likely (must further research cubespace adcs interface control document and connections. also adcs is still uncertain)\n"
 		(exclude_from_sim no)
 		(at 413.258 384.048 0)
@@
 		)
 	)
+	(text "Not Sure if this is how rs422 is implemented or if it works\nthis way. Must look into deeply first"
+		(exclude_from_sim no)
+		(at 537.21 528.066 0)
+		(effects
+			(font
+				(size 1.27 1.27)
+			)
+		)
+	)
 	(text "i2c and rs422"
 		(exclude_from_sim no)
@@
 	(text "Board Power Monitor"
 		(exclude_from_sim no)
-		(at 633.984 275.59 0)
+		(at 648.462 272.288 0)
 		(effects
 			(font
-				(size 1.778 1.778)
+				(size 2.032 2.032)
 				(thickness 0.3556)
 				(bold yes)
@@
 		)
 	)
-	(text "assign pin for output"
+	(text "assign pin for output (likely to load switch\n to onboard power regulators/power \nload switch that allows for power cycling)"
 		(exclude_from_sim no)
-		(at 307.594 520.7 0)
+		(at 316.23 525.272 0)
 		(effects
 			(font
@@
 		)
 	)
-	(text "gonna nuke eeprom (nominally more likely to be affected by radiation)\nkeeping for now in case mind changes"
+	(text "prob gonna nuke eeprom (nominally more likely to be affected by radiation)\nkeeping for now in case mind changes"
 		(exclude_from_sim no)
 		(at 413.766 520.7 0)
@@
 	(text "put boxes randomly around for now,\nwill move to separate sheets later.\n-William"
 		(exclude_from_sim no)
-		(at 395.478 496.062 0)
+		(at 659.638 559.562 0)
 		(effects
 			(font
@@
 		)
 	)
+	(text "rs422 prob doesnt work this way. look into implementation and\nif we can use uart to rs422 or if we need dedicated ftdi chip or something"
+		(exclude_from_sim no)
+		(at 572.262 471.424 0)
+		(effects
+			(font
+				(size 1.27 1.27)
+			)
+		)
+	)
 	(text "I2C Address: 1000000"
 		(exclude_from_sim no)
@@
 		)
 	)
+	(text "VBATT-->Regulator_Output-->3.3V"
+		(exclude_from_sim no)
+		(at 706.628 228.346 0)
+		(effects
+			(font
+				(size 1.7018 1.7018)
+				(thickness 0.3404)
+				(bold yes)
+			)
+		)
+	)
 	(text "WDT enabled\nwhen soldered"
 		(exclude_from_sim no)
@@
 		)
 	)
-	(text "TO DO:\n- assign i2c addresses to power monitors\n- reorganize board to board connections\n- double check memory implementations (ospi left now)\n- add heater and antenna trigger\n- add more watchdogs (for power, processor, satnogs)\n-assign watchdog input/output pins\n-add rs422 transceiver to payload connection\n"
+	(text "TO DO:\n- reorganize & fully implement board to board connections (SATNOGS should only need i2c now but double check; payload needs few i2c bus and rs422 if possible;adcs connection needs to be implemented)\n- double check octal spi nor flash memory implementation (very briefly skimmed datasheet)\n- add heater and antenna trigger connection/connector (need to talk with thermals & power about interface)\n- add more watchdog (for onboard power, satnogs)\n-assign watchdog input/output pins (pet pins, destination of outputs)\n-implement watchdog bite power cycling \n(load switch powering off processor briefly to force reset in case of radiation event)\n-add rs422 transceiver to payload connection/if possible\n-look into coin batteries for skytraq gnss and imx8x som (while also making sure safe in space)\n-connect RTC"
 		(exclude_from_sim no)
-		(at 473.456 431.292 0)
+		(at 464.566 440.436 0)
 		(effects
 			(font
@@
 	(global_label "X_UART1_CTS_B"
 		(shape input)
-		(at 622.3 482.6 180)
+		(at 530.86 516.89 180)
 		(effects
 			(font
@@
 		)
 		(property "Intersheetrefs" "${INTERSHEET_REFS}"
-			(at 622.3 482.6 0)
+			(at 530.86 516.89 0)
 			(effects
 				(font
@@
 	(global_label "X_UART1_RTS_B"
 		(shape output)
-		(at 622.3 485.14 180)
+		(at 530.86 519.43 180)
 		(effects
 			(font
@@
 		)
 		(property "Intersheetrefs" "${INTERSHEET_REFS}"
-			(at 622.3 485.14 0)
+			(at 530.86 519.43 0)
 			(effects
 				(font

Commit message: more notes
Other:
- note added: "might have to put one or two more watchdogs (satnogs and power board) requires more research into satnogs fault tolerance/onboard capabilities while power board requires more discussion with power team"
Changed lines of the file:
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@@
 	(text "add i2c line to satnogs connection"
 		(exclude_from_sim no)
-		(at 772.16 479.806 0)
+		(at 776.986 479.806 0)
 		(effects
 			(font
@@
 			)
 		)
+	)
+	(text "might have to put one or two more watchdogs (satnogs and power board)\nrequires more research into satnogs fault tolerance/onboard capabilities while\npower board requires more discussion with power team"
+		(exclude_from_sim no)
+		(at 209.804 566.166 0)
+		(effects
+			(font
+				(size 3.048 3.048)
+				(thickness 0.6096)
+				(bold yes)
+			)
+		)

Commit message: fixed connection with uart label
Parts:
- added CN3: DF11-16DP-2DSA(08), imx8_carrier_board_footprints:CONN-TH_DF11-16DP-2DSA-08, symbol cadence imx8_carrier_board_symbol_library:DF11-16DP-2DSA(08)
Connections:
- net M40_UART0_TX (Watchdog Pet): no longer J?.C62 (X_SCU_GPIO0_01)
- net M40_UART0_RX renamed X_M40_UART0_RX
- new net X_M40_UART0_TX: J?.C62 (X_SCU_GPIO0_01)
Other:
- note added: "Ebyte RF Transceiver Connection"
Changed lines of the file:
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@@
 		)
 	)
+	(text "Ebyte RF Transceiver Connection"
+		(exclude_from_sim no)
+		(at 719.582 208.788 0)
+		(effects
+			(font
+				(size 1.27 1.27)
+			)
+		)
+	)
 	(text "Skytraq Orion B16 UART GPS Module & Power Monitor"
 		(exclude_from_sim no)
@@
 	(text "VBATT-->Regulator_Output-->3.3V"
 		(exclude_from_sim no)
-		(at 706.628 228.346 0)
+		(at 637.286 234.696 0)
 		(effects
 			(font
@@
 		)
 	)
-	(global_label "M40_UART0_TX (Watchdog Pet)"
+	(global_label "X_M40_UART0_TX"
 		(shape bidirectional)
 		(at 308.61 194.31 180)
@@
 		)
 	)
-	(global_label "M40_UART0_RX"
+	(global_label "X_M40_UART0_RX"
 		(shape bidirectional)
 		(at 308.61 191.77 180)
@@
 					(unit 1)
 				)
+			)
+		)
+	)
+	(symbol
+		(lib_id "cadence imx8_carrier_board_symbol_library:DF11-16DP-2DSA(08)")
+		(at 718.82 229.87 0)
+		(unit 1)
+		(exclude_from_sim no)
+		(in_bom yes)
+		(on_board yes)
+		(dnp no)
+		(fields_autoplaced yes)
+		(property "Reference" "CN3"
+			(at 718.82 213.36 0)
+			(effects
+				(font
+					(size 1.27 1.27)
+				)
+			)
+		)
+		(property "Value" "DF11-16DP-2DSA(08)"
+			(at 718.82 215.9 0)
+			(effects
+				(font
+					(size 1.27 1.27)
+				)
+			)
+		)
+		(property "Footprint" "imx8_carrier_board_footprints:CONN-TH_DF11-16DP-2DSA-08"
+			(at 718.82 246.38 0)
+			(effects
+				(font
+					(size 1.27 1.27)
+				)
+				(hide yes)
+			)
+		)
+		(property "Datasheet" "https://lcsc.com/product-detail/Wire-To-Board-Wire-To-Wire-Connector_HRS-Hirose-HRS-DF11-16DP-2DSA-08_C530981.html"
+			(at 718.82 248.92 0)
+			(effects
+				(font
+					(size 1.27 1.27)
+				)
+				(hide yes)
+			)
+		)
+		(property "Description" "DF11 Connector"
+			(at 718.82 229.87 0)
+			(effects
+				(font
+					(size 1.27 1.27)
+				)
+				(hide yes)
+			)
+		)
+		(property "LCSC Part" "C530981"
+			(at 718.82 251.46 0)
+			(effects
+				(font
+					(size 1.27 1.27)
+				)
+				(hide yes)
+			)
+		)
+		(pin "14"
+		)
+		(pin "1"
+		)
+		(pin "12"
+		)
+		(pin "6"
+		)
+		(pin "8"
+		)
+		(pin "4"
+		)
+		(pin "11"
+		)
+		(pin "13"
+		)
+		(pin "10"
+		)
+		(pin "7"
+		)
+		(pin "3"
+		)
+		(pin "16"
+		)
+		(pin "2"
+		)
+		(pin "5"
+		)
+		(pin "15"
+		)
+		(pin "9"
+		)
+		(instances
+			(project "CADENCE i.MX8X Carrier Board rev1"
+				(path "/de284495-d382-47cb-b528-76e440980d40/f5f49c98-aaea-4f03-a1b3-a277d1d06600"
+					(reference "CN3")
+					(unit 1)
+				)

Commit message: Sheet Organization
Parts:
- removed C1, C2, C5, C55, C58, C61, C62, C84, C85, C86, C9, C?: 100nF, symbol Device:C
- removed C3, C4, C57, C6, C7, C8: 10u, symbol Device:C
- removed C39, C40, C41, C42, C43: 10uF, Capacitor_SMD:C_0603_1608Metric, symbol Device:C_Small
- removed C56: 220nF, symbol Device:C
- removed C87: 10uF, symbol Device:C
- removed CN1, CN2, CN3: DF11-16DP-2DSA(08), imx8_carrier_board_footprints:CONN-TH_DF11-16DP-2DSA-08, symbol cadence imx8_carrier_board_symbol_library:DF11-16DP-2DSA(08)
- removed D12: GREEN, LED_SMD:LED_0603_1608Metric, symbol Device:LED_Small_Filled
- removed D13: 1N4151WS, Diode_SMD:D_SOD-323, symbol oresat-diodes:1N4151WS-HE3
- removed J1: Micro_SD_Card_Det1, symbol Connector:Micro_SD_Card_Det1
- removed J12: Conn_01x02, Connector_PinHeader_2.54mm:PinHeader_1x02_P2.54mm_Vertical, symbol Connector_Generic:Conn_01x02
- removed J2: USB_A, symbol Connector:USB_A
- removed J3: Conn_Coaxial, symbol Connector:Conn_Coaxial
- removed J4, J9: Conn_02x26_Odd_Even, symbol Connector_Generic:Conn_02x26_Odd_Even
- removed J7: Conn_02x06_Odd_Even, symbol Connector_Generic:Conn_02x06_Odd_Even
- removed J?: USB_C_Receptacle_USB2.0_16P, symbol Connector:USB_C_Receptacle_USB2.0_16P
- removed JP1: SolderJumper_2_Open, Jumper:SolderJumper-2_P1.3mm_Open_RoundedPad1.0x1.5mm, symbol Jumper:SolderJumper_2_Open
- removed R1, R104, R105, R106, R6, R7: 49.9k, symbol Device:R
- removed R100, R101, R2, R64, R65, R98, R99, R?: 10k, symbol Device:R
- removed R107, R108, R109, R110, R111: 22, symbol Device:R
- removed R12, R3: 0.002, symbol Device:R
- removed R25, R26, R27, R31, R32: 10k, Resistor_SMD:R_0603_1608Metric, symbol Device:R_Small_US
- removed R28, R29, R30: 3.0k, Resistor_SMD:R_0603_1608Metric, symbol Device:R_Small_US
- removed R33, R35: 1k, Resistor_SMD:R_0603_1608Metric, symbol Device:R_Small_US
- removed R34, R36, R37, R38, R40: 100k, Resistor_SMD:R_0603_1608Metric, symbol Device:R_Small_US
- removed R39: 4.7M, Resistor_SMD:R_0603_1608Metric, symbol Device:R_Small_US
- removed R8, R9: 5.1k, symbol Device:R
- removed SW1: SW_DIP_x04, symbol Switch:SW_DIP_x04
- removed TP11, TP12, TP13, TP14, TP15: TestPoint-MinTH, oresat-misc:TestPoint-0.75mm-th, symbol oresat-misc:Test-Point-0.75mm-th
- removed U1, U2: INA219AxDCN, Package_TO_SOT_SMD:SOT-23-8, symbol Sensor_Energy:INA219AxDCN
- removed U10, U14: MR20H40, symbol Memory_NVRAM:MR20H40
- removed U11: LSM6DSO, symbol cadence carrier custom symbols:LSM6DSO
- removed U12: LIS2MDL, Package_LGA:LGA-12_2x2mm_P0.5mm, symbol Sensor_Magnetic:LIS2MDL
- removed U15: TLV1704, Package_SO:TSSOP-14_4.4x5mm_P0.65mm, symbol oresat-ics:TLV1704AIPWR
- removed U20: ZDSD04GLGEAG, symbol cadence carrier custom symbols:ZDSD04GLGEAG
- removed U24: TMP112xxDRL, Package_TO_SOT_SMD:SOT-563, symbol Sensor_Temperature:TMP112xxDRL
- removed U29, U30: USBLC6-2SC6, Package_TO_SOT_SMD:SOT-23-6, symbol Power_Protection:USBLC6-2SC6
- removed U3, U32, U4: P82B715DR, symbol cadence carrier custom symbols:TI_P82B715DR
- removed U31: MAX3485, Package_SO:SOIC-8_3.9x4.9mm_P1.27mm, symbol Interface_UART:MAX3485
- removed U6: Skytraq Orion B16 GPS, symbol skytraq_orion_b16_gps:Skytraq_Orion_B16_GPS
- removed U7, U8: AMS1117-3.3, Package_TO_SOT_SMD:SOT-223-3_TabPin2, symbol Regulator_Linear:AMS1117-3.3
- removed U9: RV-3028-C7, Package_SON:MicroCrystal_C7_SON-8_1.5x3.2mm_P0.9mm, symbol Timer_RTC:RV-3028-C7
- removed U?: MX25UM51245G, symbol cadence carrier custom symbols:MX25UM51245G
- removed U?: 25CSM04xxSN, Package_SO:SOIC-8_3.9x4.9mm_P1.27mm, symbol Memory_EEPROM:25CSM04xxSN
Connections:
- no-connect marks 103 -> 0
Other:
- note removed: "4Mbit (0.5MB), $30 a unit"
- note removed: "4Mbit EEPROM (0.5MB)"
- note removed: "512 Mbit (64MB) NOR Flash (Important Telemetry/ slightly less critical info)"
- note removed: "5v to 3.3v regulators (1A output each IC)"
- note removed: "ADCS? Connection"
- note removed: "Accelerometer & Gyroscope"
- note removed: "Battery Board Connection"
- note removed: "Board Power Monitor"
- note removed: "Boot Mode Control"
- note removed: "D5 and D7 MUST be 1N4151WS"
- note removed: "DC block and pulse detector"
- note removed: "Disable shutdown during initial power up."
- note removed: "Do Not Consolidate the BOM on this Circuit"
- note removed: "Ebyte RF Transceiver Connection"
- note removed: "External Board Connections"
- note removed: "External Watch-Dog Timer"
- note removed: "I2C Address: 0011110b"
- note removed: "I2C Address: 1000000"
- note removed: "I2C Address: 1000100"
- note removed: "I2C Address: 1001000"
- note removed: "I2C Address: 1010010b"
- note removed: "I2C Address: 1101010b"
- note removed: "IMU (Accelerometer, Gyroscope, Magnetometer)"
- note removed: "List of Power Monitors: - x1 Overall Power Monitor - x1 GNSS Power Monitor - x1"
- note removed: "MR25H40MDF"
- note removed: "MRAM (important/critical data)"
- note removed: "Magnetometer"
- note removed: "NAND Flash (Images/Non critical info)"
- note removed: "Not Required if Power is Not Crowbarred"
- note removed: "Not Sure if this is how rs422 is implemented or if it works this way. Must look into deeply first"
- note removed: "Oscillator"
- note removed: "Output buffer"
- note removed: "Payload Board Connection"
- note removed: "Pull-up on battery pack to Vbus"
- note removed: "Pulse integrator"
- note removed: "RTC (real time clock) module (i2c or spi)"
- note removed: "SATNOGS Board Connection"
- note removed: "SPI0 Bus"
- note removed: "Select 15V-25V on C36, C37, C38, C39"
- note removed: "Skytraq Orion B16 UART GPS Module & Power Monitor"
- note removed: "TLV1704AMPWPSEP is the radiation tolerant version. Use TLV1704AQPWRQ1 for non-flight C3 boards."
- note removed: "Temperature Sensor"
- note removed: "USB Ports (for debug, coding, development)"
- note removed: "VBATT-->Regulator_Output-->3.3V"
- note removed: "WDT enabled when soldered"
- note removed: "Watchdog based upon PROVES FC V5's & Oresat's C3 Board"
- note removed: "ZDSD04GLGEAG"
- note removed: "add i2c line to satnogs connection"
- note removed: "assign pin for output (likely to load switch to onboard power regulators/power load switch that allows for power cycling)"
- note removed: "assign pin for watchdog pet"
- note removed: "connect to gpio for reset signal"
- note removed: "connect to gpio on imx (1pps) maybe also add bootsel?"
- note removed: "connector h1"
- note removed: "connector h2"
- note removed: "df11 interim connector used"
- note removed: "https://www.digikey.com/en/products/detail/everspin-technologies-inc/MR20H40CDF/4047456"
- note removed: "i2c and rs422"
- note removed: "less susceptible to radiation effects (less FETs per bit)"
- note removed: "microSD"
- note removed: "might have to put one or two more watchdogs (satnogs and power board) requires more research into satnogs fault tolerance/onboard capabilities while power board requires more discussion with power team"
- note removed: "prob gonna nuke eeprom (nominally more likely to be affected by radiation) keeping for now in case mind changes"
- note removed: "rs422 prob doesnt work this way. look into implementation and if we can use uart to rs422 or if we need dedicated ftdi chip or something"
- note removed: "usb termination resistor values may be changed to adjust impedance"
- note removed: "~ 24 s period (36 s on power up)"
