File: hardware/i.MX8X Flight Computer Carrier Board/CADENCE i.MX8X Carrier Board rev1/Flash.kicad_sch (KiCad schematic)
At the start: 12 parts, among them U10 MR20H40, U11 MR20H40, U8 MX25UM51245G, U9 ZDSD04GLGEAG

Commit message: final rev1 schematic changes for phytec
Connections:
- net X_MIPI_CSI0_GPIO0_00 renamed X_FLEXCAN1_RX (GPIO)
Other:
- note added: "1.8V GPIO"
Changed lines of the file:
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@@
+		)
+	)
+	(text "1.8V GPIO"
+		(exclude_from_sim no)
+		(at 110.998 63.5 0)
+		(effects
+			(font
+				(size 1.27 1.27)
+			)
 		)
 	)
@@
 		)
 	)
-	(global_label "X_MIPI_CSI0_GPIO0_00"
-		(shape bidirectional)
-		(at 102.87 66.04 0)
-		(effects
-			(font
-				(size 1.27 1.27)
-			)
-			(justify left)
-		)
-		(property "Intersheetrefs" "${INTERSHEET_REFS}"
-			(at 102.87 66.04 0)
-			(effects
-				(font
-					(size 1.27 1.27)
-				)
-				(hide yes)
-			)
-		)
-	)
 	(global_label "X_QSPI0_DATA6"
 		(shape bidirectional)
@@
 		(property "Intersheetrefs" "${INTERSHEET_REFS}"
 			(at 97.79 134.62 0)
+			(effects
+				(font
+					(size 1.27 1.27)
+				)
+				(hide yes)
+			)
+		)
+	)
+	(global_label "X_FLEXCAN1_RX (GPIO)"
+		(shape bidirectional)
+		(at 102.87 66.04 0)
+		(effects
+			(font
+				(size 1.27 1.27)
+				(thickness 0.254)
+				(bold yes)
+			)
+			(justify left)
+		)
+		(property "Intersheetrefs" "${INTERSHEET_REFS}"
+			(at 102.87 66.04 0)
 			(effects
 				(font
@@
 		(dnp no)
 		(fields_autoplaced yes)
-		(property "Reference" "#PWR059"
+		(property "Reference" "#PWR061"
 			(at 104.14 124.46 0)
 			(effects
@@
 			(project "CADENCE i.MX8X Carrier Board rev1"
 				(path "/de284495-d382-47cb-b528-76e440980d40/711a63dc-df49-4577-a994-dfb9f7680289"
-					(reference "#PWR059")
+					(reference "#PWR061")
 					(unit 1)
 				)
@@
 		(on_board yes)
 		(dnp no)
-		(property "Reference" "#PWR057"
+		(property "Reference" "#PWR059"
 			(at 100.33 59.69 0)
 			(effects
@@
 			(project "CADENCE i.MX8X Carrier Board rev1"
 				(path "/de284495-d382-47cb-b528-76e440980d40/711a63dc-df49-4577-a994-dfb9f7680289"
-					(reference "#PWR057")
+					(reference "#PWR059")
 					(unit 1)
 				)
@@
 		(dnp no)
 		(fields_autoplaced yes)
-		(property "Reference" "#PWR056"
+		(property "Reference" "#PWR058"
 			(at 62.23 152.4 0)
 			(effects
@@
 			(project "CADENCE i.MX8X Carrier Board rev1"
 				(path "/de284495-d382-47cb-b528-76e440980d40/711a63dc-df49-4577-a994-dfb9f7680289"
-					(reference "#PWR056")
+					(reference "#PWR058")
 					(unit 1)
 				)
@@
 		(on_board yes)
 		(dnp no)
-		(property "Reference" "#PWR062"
+		(property "Reference" "#PWR064"
 			(at 194.31 109.22 0)
 			(effects
@@
 			(project "CADENCE i.MX8X Carrier Board rev1"
 				(path "/de284495-d382-47cb-b528-76e440980d40/711a63dc-df49-4577-a994-dfb9f7680289"
-					(reference "#PWR062")
+					(reference "#PWR064")
 					(unit 1)
 				)
@@
 		(dnp no)
 		(fields_autoplaced yes)
-		(property "Reference" "#PWR061"
+		(property "Reference" "#PWR063"
 			(at 194.31 97.79 0)
 			(effects
@@
 			(project "CADENCE i.MX8X Carrier Board rev1"
 				(path "/de284495-d382-47cb-b528-76e440980d40/711a63dc-df49-4577-a994-dfb9f7680289"
-					(reference "#PWR061")
+					(reference "#PWR063")
 					(unit 1)
 				)
@@
 		(dnp no)
 		(fields_autoplaced yes)
-		(property "Reference" "#PWR063"
+		(property "Reference" "#PWR065"
 			(at 194.31 139.7 0)
 			(effects
@@
 			(project "CADENCE i.MX8X Carrier Board rev1"
 				(path "/de284495-d382-47cb-b528-76e440980d40/711a63dc-df49-4577-a994-dfb9f7680289"
-					(reference "#PWR063")
+					(reference "#PWR065")
 					(unit 1)
 				)
@@
 		(dnp no)
 		(fields_autoplaced yes)
-		(property "Reference" "#PWR058"
+		(property "Reference" "#PWR060"
 			(at 100.33 92.71 0)
 			(effects
@@
 			(project "CADENCE i.MX8X Carrier Board rev1"
 				(path "/de284495-d382-47cb-b528-76e440980d40/711a63dc-df49-4577-a994-dfb9f7680289"
-					(reference "#PWR058")
+					(reference "#PWR060")
 					(unit 1)
 				)
@@
 		(on_board yes)
 		(dnp no)
-		(property "Reference" "#PWR060"
+		(property "Reference" "#PWR062"
 			(at 194.31 66.04 0)
 			(effects
@@
 			(project "CADENCE i.MX8X Carrier Board rev1"
 				(path "/de284495-d382-47cb-b528-76e440980d40/711a63dc-df49-4577-a994-dfb9f7680289"
-					(reference "#PWR060")
+					(reference "#PWR062")
 					(unit 1)
 				)

Commit message: updated imx8x footprints
Parts:
- U10, U11: footprint (none) -> Footprints:SON127P600X500X90-9N-D
Changed lines of the file:
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@@
 			)
 		)
-		(property "Footprint" ""
+		(property "Footprint" "Footprints:SON127P600X500X90-9N-D"
 			(at 194.31 78.74 0)
 			(effects
@@
 			)
 		)
-		(property "Footprint" ""
+		(property "Footprint" "Footprints:SON127P600X500X90-9N-D"
 			(at 194.31 120.65 0)
 			(effects

Commit message: added footprints to imx8x, just need to finish usb, capacitors, and inductors
Parts:
- C47, C48, C49, C50: footprint (none) -> Capacitor_SMD:C_0603_1608Metric
- R53, R54, R55, R56: footprint (none) -> Resistor_SMD:R_0402_1005Metric
- U8: footprint (none) -> Footprints:SOP-16_L10.3-W7.5-P1.27-LS10.3-BL
- U9: footprint (none) -> Footprints:LGA-8_L8.0-W6.0-P1.27-TL-1
Changed lines of the file:
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@@
 			)
 		)
-		(property "Footprint" ""
+		(property "Footprint" "Footprints:LGA-8_L8.0-W6.0-P1.27-TL-1"
 			(at 82.55 120.65 0)
 			(effects
@@
 			)
 		)
-		(property "Footprint" ""
+		(property "Footprint" "Capacitor_SMD:C_0603_1608Metric"
 			(at 116.5352 137.16 0)
 			(effects
@@
 			)
 		)
-		(property "Footprint" ""
+		(property "Footprint" "Footprints:SOP-16_L10.3-W7.5-P1.27-LS10.3-BL"
 			(at 81.28 53.34 0)
 			(effects
@@
 			)
 		)
-		(property "Footprint" ""
+		(property "Footprint" "Resistor_SMD:R_0402_1005Metric"
 			(at 182.118 71.12 90)
 			(effects
@@
 			)
 		)
-		(property "Footprint" ""
+		(property "Footprint" "Resistor_SMD:R_0402_1005Metric"
 			(at 182.118 114.3 90)
 			(effects
@@
 			)
 		)
-		(property "Footprint" ""
+		(property "Footprint" "Capacitor_SMD:C_0603_1608Metric"
 			(at 101.2952 77.47 0)
 			(effects
@@
 			)
 		)
-		(property "Footprint" ""
+		(property "Footprint" "Capacitor_SMD:C_0603_1608Metric"
 			(at 159.7152 125.73 0)
 			(effects
@@
 			)
 		)
-		(property "Footprint" ""
+		(property "Footprint" "Capacitor_SMD:C_0603_1608Metric"
 			(at 159.7152 82.55 0)
 			(effects
@@
 			)
 		)
-		(property "Footprint" ""
+		(property "Footprint" "Resistor_SMD:R_0402_1005Metric"
 			(at 174.498 114.3 90)
 			(effects
@@
 			)
 		)
-		(property "Footprint" ""
+		(property "Footprint" "Resistor_SMD:R_0402_1005Metric"
 			(at 173.228 72.39 90)
 			(effects

Commit message: cchanges after phytec review
- fixed issue with ospi chip select line & clk line
- replaced 1k pulldowns with 10k pulldowns and added 1k series resistors to 1.8V line for boot config lines
-removed unused global label tags from som and changed to nc
- repinmuxed for potential watchdog and ospi changes

to do:
-microSD
-reallocate gpios (extras to breakout)
-create 8pin jst connector for lucid camera (12V pwr)
- give satnogs additional uart
- reorg/rename global labels
-watchdog input pin reassign to c62 potentially after feedback from max
Parts:
- renumbered R53 to R57, R54 to R58, R55 to R59, R56 to R60
Connections:
- net X_QSPI0A_SS0_B renamed X_QSPI0A_SS1_B
- net X_QSPI0B_SCLK renamed X_QSPI0A_SCLK
Changed lines of the file:
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@@
+		)
+	)
+	(global_label "X_QSPI0A_SCLK"
+		(shape input)
+		(at 67.31 85.09 180)
+		(effects
+			(font
+				(size 1.27 1.27)
+			)
+			(justify right)
+		)
+		(property "Intersheetrefs" "${INTERSHEET_REFS}"
+			(at 67.31 85.09 0)
+			(effects
+				(font
+					(size 1.27 1.27)
+				)
+				(hide yes)
+			)
 		)
 	)
@@
 		)
 	)
+	(global_label "X_QSPI0A_SS1_B"
+		(shape input)
+		(at 67.31 58.42 180)
+		(effects
+			(font
+				(size 1.27 1.27)
+				(thickness 0.1588)
+			)
+			(justify right)
+		)
+		(property "Intersheetrefs" "${INTERSHEET_REFS}"
+			(at 67.31 58.42 0)
+			(effects
+				(font
+					(size 1.27 1.27)
+				)
+				(hide yes)
+			)
+		)
+	)
 	(global_label "X_QSPI0_DATA2"
 		(shape bidirectional)
@@
 		)
 	)
-	(global_label "X_QSPI0A_SS0_B"
-		(shape input)
-		(at 67.31 58.42 180)
-		(effects
-			(font
-				(size 1.27 1.27)
-			)
-			(justify right)
-		)
-		(property "Intersheetrefs" "${INTERSHEET_REFS}"
-			(at 67.31 58.42 0)
-			(effects
-				(font
-					(size 1.27 1.27)
-				)
-				(hide yes)
-			)
-		)
-	)
 	(global_label "X_SPI0_SDO"
 		(shape input)
@@
 		)
 	)
-	(global_label "X_QSPI0B_SCLK"
-		(shape input)
-		(at 67.31 85.09 180)
-		(effects
-			(font
-				(size 1.27 1.27)
-			)
-			(justify right)
-		)
-		(property "Intersheetrefs" "${INTERSHEET_REFS}"
-			(at 67.31 85.09 0)
-			(effects
-				(font
-					(size 1.27 1.27)
-				)
-				(hide yes)
-			)
-		)
-	)
 	(global_label "X_SPI2_CS0"
 		(shape bidirectional)
@@
 		(on_board yes)
 		(dnp no)
-		(property "Reference" "R55"
+		(property "Reference" "R59"
 			(at 184.15 69.342 0)
 			(effects
@@
 			(project "CADENCE i.MX8X Carrier Board rev1"
 				(path "/de284495-d382-47cb-b528-76e440980d40/711a63dc-df49-4577-a994-dfb9f7680289"
-					(reference "R55")
+					(reference "R59")
 					(unit 1)
 				)
@@
 		(on_board yes)
 		(dnp no)
-		(property "Reference" "R56"
+		(property "Reference" "R60"
 			(at 184.15 112.522 0)
 			(effects
@@
 			(project "CADENCE i.MX8X Carrier Board rev1"
 				(path "/de284495-d382-47cb-b528-76e440980d40/711a63dc-df49-4577-a994-dfb9f7680289"
-					(reference "R56")
+					(reference "R60")
 					(unit 1)
 				)
@@
 		(on_board yes)
 		(dnp no)
-		(property "Reference" "R54"
+		(property "Reference" "R58"
 			(at 176.53 112.522 0)
 			(effects
@@
 			(project "CADENCE i.MX8X Carrier Board rev1"
 				(path "/de284495-d382-47cb-b528-76e440980d40/711a63dc-df49-4577-a994-dfb9f7680289"
-					(reference "R54")
+					(reference "R58")
 					(unit 1)
 				)
@@
 		(on_board yes)
 		(dnp no)
-		(property "Reference" "R53"
+		(property "Reference" "R57"
 			(at 175.26 70.612 0)
 			(effects
@@
 			(project "CADENCE i.MX8X Carrier Board rev1"
 				(path "/de284495-d382-47cb-b528-76e440980d40/711a63dc-df49-4577-a994-dfb9f7680289"
-					(reference "R53")
-					(unit 1)
-				)
+					(reference "R57")
+					(unit 1)
+				)

Commit message: imx8x som connector schematic update
-fixed the microsd implementation
-fixed an oopsie where i accidentally removed the ethernet som connections and marked as nc (2am oopsie lol),
-renamed the som global labels as their som signals
-modified watchdog input from the jtag trst to the dedicated wdog output pin on som

to do:
-breakout connectors for gpio & adc
-test/debug points/ports
- connect 1 more gpio to ebyte connection
- connect uart2 to satnogs, no longer free use as breakout
-check footprints
Connections:
- net X_FLEXCAN1_RX (GPIO) renamed LSIO_GPIO1_IO17
Changed lines of the file:
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@@
+		)
+	)
+	(global_label "LSIO_GPIO1_IO17"
+		(shape bidirectional)
+		(at 102.87 66.04 0)
+		(fields_autoplaced yes)
+		(effects
+			(font
+				(size 1.27 1.27)
+				(thickness 0.254)
+				(bold yes)
+			)
+			(justify left)
+		)
+		(property "Intersheetrefs" "${INTERSHEET_REFS}"
+			(at 123.5897 66.04 0)
+			(effects
+				(font
+					(size 1.27 1.27)
+				)
+				(justify left)
+				(hide yes)
+			)
 		)
 	)
@@
 			(effects
 				(font
-					(size 1.27 1.27)
-				)
-				(hide yes)
-			)
-		)
-	)
-	(global_label "X_FLEXCAN1_RX (GPIO)"
-		(shape bidirectional)
-		(at 102.87 66.04 0)
-		(effects
-			(font
-				(size 1.27 1.27)
-				(thickness 0.254)
-				(bold yes)
-			)
-			(justify left)
-		)
-		(property "Intersheetrefs" "${INTERSHEET_REFS}"
-			(at 102.87 66.04 0)
-			(effects
-				(font

Commit message: reorged pin definitions page
Connections:
- net LSIO_GPIO1_IO17 renamed LSIO_GPIO3_IO14
Changed lines of the file:
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@@
+		)
+	)
+	(global_label "LSIO_GPIO3_IO14"
+		(shape bidirectional)
+		(at 102.87 66.04 0)
+		(effects
+			(font
+				(size 1.27 1.27)
+				(thickness 0.254)
+				(bold yes)
+			)
+			(justify left)
+		)
+		(property "Intersheetrefs" "${INTERSHEET_REFS}"
+			(at 102.87 66.04 0)
+			(effects
+				(font
+					(size 1.27 1.27)
+				)
+				(hide yes)
+			)
 		)
 	)
@@
 				(hide yes)
 			)
-		)
-	)
-	(global_label "LSIO_GPIO1_IO17"
-		(shape bidirectional)
-		(at 102.87 66.04 0)
-		(fields_autoplaced yes)
-		(effects
-			(font
-				(size 1.27 1.27)
-				(thickness 0.254)
-				(bold yes)
-			)
-			(justify left)
-		)
-		(property "Intersheetrefs" "${INTERSHEET_REFS}"
-			(at 123.5897 66.04 0)
-			(effects
-				(font
-					(size 1.27 1.27)
-				)
-				(justify left)
-				(hide yes)
-			)

Commit message: Finished footprints- Double check usbs
Only thing i didn't touch was watchdogs. That might still need to be changed.
Parts:
- C47, C48, C49, C50: footprint Capacitor_SMD:C_0603_1608Metric -> Capacitor_SMD:C_0402_1005Metric
Changed lines of the file:
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@@
 			)
 		)
-		(property "Footprint" "Capacitor_SMD:C_0603_1608Metric"
+		(property "Footprint" "Capacitor_SMD:C_0402_1005Metric"
 			(at 116.5352 137.16 0)
 			(effects
@@
 			)
 		)
-		(property "Footprint" "Capacitor_SMD:C_0603_1608Metric"
+		(property "Footprint" "Capacitor_SMD:C_0402_1005Metric"
 			(at 101.2952 77.47 0)
 			(effects
@@
 			)
 		)
-		(property "Footprint" "Capacitor_SMD:C_0603_1608Metric"
+		(property "Footprint" "Capacitor_SMD:C_0402_1005Metric"
 			(at 159.7152 125.73 0)
 			(effects
@@
 			)
 		)
-		(property "Footprint" "Capacitor_SMD:C_0603_1608Metric"
+		(property "Footprint" "Capacitor_SMD:C_0402_1005Metric"
 			(at 159.7152 82.55 0)
 			(effects

Commit message: connection changes, debug headers, fixing critical issues
-finished debug/utility header pin section (may have to reassign some gpios again tho)
- added can bus transceiver and connection to satnogs
- reassigned/ ensured no i2c address conflict
- resolved critical error in LTC-3115 power regulator symbol where output power was shorted to sync pin
-resolved critical symbol issue in which imx8x som power good symbol shorted to gnd, which would result in nonfunctional board & 2 jtag pins shorted

to do:
- assign gpio to a load switch
- resolve erc issues
- footprint check (shunt resistor change, some new ics need footprints, cmos image sensor 8 pin jst connector, etc)
Parts:
- added TP22: TestPoint, TestPoint:TestPoint_Pad_1.0x1.0mm, symbol EPS:TestPoint
Connections:
- net P_1V8_OUT: now also TP22.1
Other:
- note removed: "MR25H40MDF"
Changed lines of the file:
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@@
-		)
-	)
-	(text "MR25H40MDF"
-		(exclude_from_sim no)
-		(at 195.834 31.496 0)
-		(effects
-			(font
-				(size 1.27 1.27)
-			)
 		)
 	)
@@
 					(unit 1)
 				)
+			)
+		)
+	)
+	(symbol
+		(lib_id "EPS:TestPoint")
+		(at 100.33 57.15 270)
+		(unit 1)
+		(exclude_from_sim no)
+		(in_bom yes)
+		(on_board yes)
+		(dnp no)
+		(property "Reference" "TP22"
+			(at 105.156 57.15 90)
+			(effects
+				(font
+					(size 1.27 1.27)
+				)
+				(justify left)
+			)
+		)
+		(property "Value" "TestPoint"
+			(at 105.41 58.4199 90)
+			(effects
+				(font
+					(size 1.27 1.27)
+				)
+				(justify left)
+				(hide yes)
+			)
+		)
+		(property "Footprint" "TestPoint:TestPoint_Pad_1.0x1.0mm"
+			(at 100.33 62.23 0)
+			(effects
+				(font
+					(size 1.27 1.27)
+				)
+				(hide yes)
+			)
+		)
+		(property "Datasheet" "~"
+			(at 100.33 62.23 0)
+			(effects
+				(font
+					(size 1.27 1.27)
+				)
+				(hide yes)
+			)
+		)
+		(property "Description" "test point"
+			(at 100.33 57.15 0)
+			(effects
+				(font
+					(size 1.27 1.27)
+				)
+				(hide yes)
+			)
+		)
+		(pin "1"
+		)
+		(instances
+			(project "CADENCE i.MX8X Carrier Board rev1"
+				(path "/de284495-d382-47cb-b528-76e440980d40/711a63dc-df49-4577-a994-dfb9f7680289"
+					(reference "TP22")
+					(unit 1)
+				)
