File: hardware/i.MX8X Flight Computer Carrier Board/CADENCE i.MX8X Carrier Board rev1/pinmux.kicad_sch (KiCad schematic)
At the start: 0 parts

Commit message: reorged pin definitions page
Other:
- note added: "Reference Page"
Changed lines of the file:
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@@
 	(generator_version "9.0")
 	(paper "A3")
+	(text "Reference\nPage"
+		(exclude_from_sim no)
+		(at 378.46 28.702 0)
+		(effects
+			(font
+				(size 6.35 6.35)
+				(thickness 1.27)
+				(bold yes)
+			)
+		)
+	)
 	(image
 		(at 140.208 148.336)
