File: hardware/i.MX8X Flight Computer Carrier Board/CADENCE i.MX8X Carrier Board rev1/FTDI.kicad_sch (KiCad schematic)
At the start: 86 parts, among them J6 USB_C_Receptacle_USB2.0_16P, Q3 BSS138, SW4 SW_DIP_x01, U30 LP38693MP-ADJ/NOPB, U31 74CBTLV3257BQ, U32 USBLC6-2SC6, U33 CAT93C66VI-GT3, U34 FT2232HL, Y2 12MHz

Commit message: added footprints to imx8x, just need to finish usb, capacitors, and inductors
Parts:
- R123, R124, R125, R126: footprint (none) -> Resistor_SMD:R_0402_1005Metric
- SW4: footprint (none) -> Footprints:SW-SMD_1.27-1P-TPPT
Changed lines of the file:
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@@
 			)
 		)
-		(property "Footprint" ""
+		(property "Footprint" "Footprints:SW-SMD_1.27-1P-TPPT"
 			(at 62.23 157.48 0)
 			(effects
@@
 			)
 		)
-		(property "Footprint" ""
+		(property "Footprint" "Resistor_SMD:R_0402_1005Metric"
 			(at 196.85 50.038 90)
 			(effects
@@
 			)
 		)
-		(property "Footprint" ""
+		(property "Footprint" "Resistor_SMD:R_0402_1005Metric"
 			(at 196.85 42.418 90)
 			(effects
@@
 			)
 		)
-		(property "Footprint" ""
+		(property "Footprint" "Resistor_SMD:R_0402_1005Metric"
 			(at 196.85 52.578 90)
 			(effects
@@
 			)
 		)
-		(property "Footprint" ""
+		(property "Footprint" "Resistor_SMD:R_0402_1005Metric"
 			(at 196.85 39.878 90)
 			(effects

Commit message: cchanges after phytec review
- fixed issue with ospi chip select line & clk line
- replaced 1k pulldowns with 10k pulldowns and added 1k series resistors to 1.8V line for boot config lines
-removed unused global label tags from som and changed to nc
- repinmuxed for potential watchdog and ospi changes

to do:
-microSD
-reallocate gpios (extras to breakout)
-create 8pin jst connector for lucid camera (12V pwr)
- give satnogs additional uart
- reorg/rename global labels
-watchdog input pin reassign to c62 potentially after feedback from max
Parts:
- renumbered C103 to C104, C104 to C105, C105 to C106, C106 to C107, C107 to C108, C108 to C109, C109 to C110, C110 to C111, C111 to C112, C112 to C113, C113 to C114, C114 to C115, C115 to C116, C116 to C117, C117 to C118, C118 to C119, C119 to C120, C120 to C121, C121 to C122, C122 to C123, C123 to C124, C124 to C125, C125 to C126, R116 to R120, R117 to R121, R118 to R122, R119 to R123, R120 to R124, R121 to R125, R122 to R126, R123 to R127, R124 to R128, R125 to R129, R126 to R130, R127 to R131, R128 to R132, R129 to R133, R130 to R134, R131 to R135, R132 to R136, R133 to R137, R134 to R138, R135 to R139, R136 to R140, R137 to R141, R138 to R142, R139 to R143, R140 to R144, R141 to R145, R142 to R146, R143 to R147, R144 to R148, R145 to R149, R146 to R150, R147 to R151, R148 to R152, R149 to R153, R150 to R154, R151 to R155, R152 to R156, R153 to R157, R154 to R158, R155 to R159, R156 to R160, R157 to R161, R158 to R162, R159 to R163, R160 to R164, R161 to R165, R162 to R166, R163 to R167, R164 to R168

Commit message: Finished footprints- Double check usbs
Only thing i didn't touch was watchdogs. That might still need to be changed.
Parts:
- C105, C106, C107, C109, C110, C112, C113, C114, C118, C120, C121, C122, C124, C126: footprint Capacitor_SMD:C_0603_1608Metric -> Capacitor_SMD:C_0402_1005Metric
- J6: footprint (none) -> Footprints:GCT_USB4085-GF-A_REVA4
Changed lines of the file:
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@@
 			)
 		)
-		(property "Footprint" "Capacitor_SMD:C_0603_1608Metric"
+		(property "Footprint" "Capacitor_SMD:C_0402_1005Metric"
 			(at 205.74 175.26 0)
 			(effects
@@
 			)
 		)
-		(property "Footprint" "Capacitor_SMD:C_0603_1608Metric"
+		(property "Footprint" "Capacitor_SMD:C_0402_1005Metric"
 			(at 328.93 173.99 0)
 			(effects
@@
 			)
 		)
-		(property "Footprint" "Capacitor_SMD:C_0603_1608Metric"
+		(property "Footprint" "Capacitor_SMD:C_0402_1005Metric"
 			(at 80.01 161.29 0)
 			(effects
@@
 			)
 		)
-		(property "Footprint" "Capacitor_SMD:C_0603_1608Metric"
+		(property "Footprint" "Capacitor_SMD:C_0402_1005Metric"
 			(at 121.92 111.76 0)
 			(effects
@@
 			)
 		)
-		(property "Footprint" "Capacitor_SMD:C_0603_1608Metric"
+		(property "Footprint" "Capacitor_SMD:C_0402_1005Metric"
 			(at 168.91 116.84 0)
 			(effects
@@
 			)
 		)
-		(property "Footprint" "Capacitor_SMD:C_0603_1608Metric"
+		(property "Footprint" "Capacitor_SMD:C_0402_1005Metric"
 			(at 101.6 184.15 0)
 			(effects
@@
 			)
 		)
-		(property "Footprint" "Capacitor_SMD:C_0603_1608Metric"
+		(property "Footprint" "Capacitor_SMD:C_0402_1005Metric"
 			(at 259.08 175.26 0)
 			(effects
@@
 			)
 		)
-		(property "Footprint" ""
+		(property "Footprint" "Footprints:GCT_USB4085-GF-A_REVA4"
 			(at 165.1 48.26 0)
 			(effects
@@
 			)
 		)
-		(property "Footprint" "Capacitor_SMD:C_0603_1608Metric"
+		(property "Footprint" "Capacitor_SMD:C_0402_1005Metric"
 			(at 367.03 173.99 0)
 			(effects
@@
 			)
 		)
-		(property "Footprint" "Capacitor_SMD:C_0603_1608Metric"
+		(property "Footprint" "Capacitor_SMD:C_0402_1005Metric"
 			(at 41.91 104.14 0)
 			(effects
@@
 			)
 		)
-		(property "Footprint" "Capacitor_SMD:C_0603_1608Metric"
+		(property "Footprint" "Capacitor_SMD:C_0402_1005Metric"
 			(at 194.31 175.26 0)
 			(effects
@@
 			)
 		)
-		(property "Footprint" "Capacitor_SMD:C_0603_1608Metric"
+		(property "Footprint" "Capacitor_SMD:C_0402_1005Metric"
 			(at 281.94 175.26 0)
 			(effects
@@
 			)
 		)
-		(property "Footprint" "Capacitor_SMD:C_0603_1608Metric"
+		(property "Footprint" "Capacitor_SMD:C_0402_1005Metric"
 			(at 270.51 175.26 0)
 			(effects
@@
 			)
 		)
-		(property "Footprint" "Capacitor_SMD:C_0603_1608Metric"
+		(property "Footprint" "Capacitor_SMD:C_0402_1005Metric"
 			(at 228.6 175.26 0)
 			(effects
@@
 			)
 		)
-		(property "Footprint" "Capacitor_SMD:C_0603_1608Metric"
+		(property "Footprint" "Capacitor_SMD:C_0402_1005Metric"
 			(at 180.34 175.26 0)
 			(effects

Commit message: Some ERC fixes, schematic annotations, pinmux for uSD & GPIO fixes, GPIO level shifter, footprint selection & pathway fix
component footprints for most part have been selected
going to double check again tmr
imx8x som bth samtec connector footprint needs to be adjusted as reference footprint uses each connector as individual symbol, while we have as part of one symbol (spacing between connector is important so som can fit in)
also one component didnt have part (uart mux) and havent assigned
implemented can bus interface with satnogs, moved around gpios, level shifted 8 gpios, fixed few missing connections (gps 1pps, a load switch enable gpio), resolved some erc errors/ symbol shorts, incorrect pinmux implementation around A9&10 for uSD and gpio, reannotated schematic, fixed footprint reference paths
Parts:
- renumbered C104 to C107, C105 to C108, C106 to C109, C107 to C110, C108 to C111, C109 to C112, C110 to C113, C111 to C114, C112 to C115, C113 to C116, C114 to C117, C115 to C118, C116 to C119, C117 to C120, C118 to C121, C119 to C122, C120 to C123, C121 to C124, C122 to C125, C123 to C126, C124 to C127, C125 to C128, C126 to C129, J6 to J5, R120 to R125, R121 to R126, R122 to R127, R123 to R128, R124 to R129, R125 to R130, R126 to R131, R127 to R132, R128 to R133, R129 to R134, R130 to R135, R131 to R136, R132 to R137, R133 to R138, R134 to R139, R135 to R140, R136 to R141, R137 to R142, R138 to R143, R139 to R144, R140 to R145, R141 to R146, R142 to R147, R143 to R148, R144 to R149, R145 to R150, R146 to R151, R147 to R152, R148 to R153, R149 to R154, R150 to R155, R151 to R156, R152 to R157, R153 to R158, R154 to R159, R155 to R160, R156 to R161, R157 to R162, R158 to R163, R159 to R164, R160 to R165, R161 to R166, R162 to R167, R163 to R168, R164 to R169, R165 to R170, R166 to R171, R167 to R172, R168 to R173, U30 to U31, U31 to U32, U32 to U33, U33 to U34, U34 to U35

Commit message: updated footprints
- shunt resistor for sense
footprint checks
- resolved mux footprint issue

to do:
-imx8x som footprint
Parts:
- U32: footprint SN74CBTLV3257PW:SOP65P640X120-16N -> Footprints:74CBTLV3257BQ115
Changed lines of the file:
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@@
 			)
 		)
-		(property "Footprint" "SN74CBTLV3257PW:SOP65P640X120-16N"
+		(property "Footprint" "Footprints:74CBTLV3257BQ115"
 			(at 82.55 208.28 0)
 			(effects

Commit message: FTDI started
Parts:
- removed R148, R149, R150, R151, R152, R153, R154, R155, R156, R157, R158, R161, R162, R163, R164, R165, R166, R167, R168, R169, R170, R171, R172: 10K, Resistor_SMD:R_0402_1005Metric, symbol Device:R_US
- added RN1: 4D02WGJ0103TCE, C61520:RES-ARRAY-SMD_0402-8P-L2.0-W1.0-BL, symbol cadence imx8_carrier_board_symbol_library:4D02WGJ0103TCE
- added RN2, RN3, RN4: 16P8WGJ103T4E, C61520:RES-ARRAY-SMD_0402-16P-L4.0-W1.6-BL, symbol cadence imx8_carrier_board_symbol_library:16P8WGJ103T4E
- R146, R147: value 10K -> 22
Connections:
- net GND: now also RN1.6, RN1.7, RN1.8, RN2.10, RN2.11, RN2.12, RN2.13, RN2.14, RN2.15, RN2.16, RN2.9, RN3.10, RN3.11, RN3.12, RN3.13, RN3.14, RN4.10, RN4.11, RN4.12, RN4.13, RN4.14, RN4.15, RN4.16
- net ACBUS6: now reaches U35.33 (ACBUS6)
- net ACBUS6: now also RN2.2
- net at U35.21 (ADBUS4): now also RN1.1
- net at U35.22 (ADBUS5): now also RN1.2
- net at U35.23 (ADBUS6): now also RN1.3
- net ACBUS0: now reaches U35.26 (ACBUS0)
- net ACBUS0: now also RN2.8
- net ACBUS1: now reaches U35.27 (ACBUS1)
- net ACBUS1: now also RN2.7
- net ACBUS2: now reaches U35.28 (ACBUS2)
- net ACBUS2: now also RN2.6
- net ACBUS3: now reaches U35.29 (ACBUS3)
- net ACBUS3: now also RN2.5
- net ACBUS4: now reaches U35.30 (ACBUS4)
- net ACBUS4: now also RN2.4
- net ACBUS5: now reaches U35.32 (ACBUS5)
- net ACBUS5: now also RN2.3
- net ACBUS7: now reaches U35.34 (ACBUS7)
- net ACBUS7: now also RN2.1
- net BDBUS2: now reaches U35.40 (BDBUS2)
- net BDBUS2: now also RN3.7
- net BDBUS3: now reaches U35.41 (BDBUS3)
- net BDBUS3: now also RN3.6
- net BDBUS4: now reaches U35.43 (BDBUS4)
- net BDBUS4: now also RN3.5
- net BDBUS5: now reaches U35.44 (BDBUS5)
- net BDBUS5: now also RN3.4
- net BDBUS6: now reaches U35.45 (BDBUS6)
- net BDBUS6: now also RN3.3
- net BCBUS0: now reaches U35.48 (BCBUS0)
- net BCBUS0: now also RN4.7
- net BCBUS1: now reaches U35.52 (BCBUS1)
- net BCBUS1: now also RN4.6
- net BCBUS2: now reaches U35.53 (BCBUS2)
- net BCBUS2: now also RN4.5
- net BCBUS3: now reaches U35.54 (BCBUS3)
- net BCBUS3: now also RN4.4
- net BCBUS4: now reaches U35.55 (BCBUS4)
- net BCBUS4: now also RN4.3
- net BCBUS5: now reaches U35.57 (BCBUS5)
- net BCBUS5: now also RN4.2
- net BCBUS6: now reaches U35.58 (BCBUS6)
- net BCBUS6: now also RN4.1
- no-connect marks 15 -> 23

Commit message: peripheral & connector layout update
- finished rs-422 payload connector layout (changed footprint, package being used has around 40 left in stock at JLCPCB)
- modified memory (mram & nor flash) ic layouts & organized into layout blocks for easy placement later
- revised & reorganized gps, rtc, temp sensor, imu connections into separate layout  blocks. also moved around gps and moved peripherals into completed layout circuit block section for later placement
- changed some power monitor shunt resistor footprints so 10W or so doesnt go thru a sad 0402 resistor lol
- fixed microSD connection issues
- adjusted gps 50 ohm coax impedance connection (28 ohm trace + 22ohm resistor)
- 50 ohm impedance calculations for gps added to schematic & disclaimer for switching regulator low ripple burst mode added to power schematic page

to do:
- verify that board power monitor wont lead to reverse current driving i.mx8x and make it explode
- look further into & verify that cmos image sensor connector is correct one being used by lucid
Parts:
- renumbered R125 to R126, R126 to R127, R127 to R128, R128 to R129, R129 to R130, R130 to R131, R131 to R132, R132 to R133, R133 to R134, R134 to R135, R135 to R136, R136 to R137, R137 to R138, R138 to R139, R139 to R140, R140 to R141, R141 to R142, R142 to R143, R143 to R144, R144 to R145, R145 to R146, R146 to R147, R147 to R148, R159 to R149, R160 to R150, R173 to R151

Commit message: pcb layout block placement
- finalized mounting hole place
- ftdi layout block complete
- more ethernet layout
- connections on board
Parts:
- J5: footprint Footprints:GCT_USB4085-GF-A_REVA4 -> Footprints:USB-C_SMD-TYPE-C-31-M-12
Changed lines of the file:
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@@
 			)
 		)
-		(property "Footprint" "Footprints:GCT_USB4085-GF-A_REVA4"
+		(property "Footprint" "Footprints:USB-C_SMD-TYPE-C-31-M-12"
 			(at 165.1 48.26 0)
 			(effects
