File: hardware/CADENCE_SWANS/Payload/Payload Controller/Prototype_Payload_Controller/mram.kicad_sch (KiCad schematic)
At the start: 3 parts

Commit message: updates
Parts:
- renumbered C4 to C45, C3 to C46, U4 to U8
Changed lines of the file:
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@@
 		(dnp no)
 		(fields_autoplaced yes)
-		(property "Reference" "#PWR020"
+		(property "Reference" "#PWR0100"
 			(at 273.05 53.34 0)
 			(effects
@@
 			(project "Payload_Controller_EM"
 				(path "/866a965d-c307-40b7-9977-69e77fc0dc82/3853f2b5-b86c-4f53-9549-ed8b814cc447"
-					(reference "#PWR020")
+					(reference "#PWR0100")
 					(unit 1)
 				)
@@
 		(on_board yes)
 		(dnp no)
-		(property "Reference" "U4"
+		(property "Reference" "U8"
 			(at 38.862 109.474 0)
 			(effects
@@
 			(project "Payload_Controller_EM"
 				(path "/866a965d-c307-40b7-9977-69e77fc0dc82/3853f2b5-b86c-4f53-9549-ed8b814cc447"
-					(reference "U4")
+					(reference "U8")
 					(unit 2)
 				)
@@
 		(dnp no)
 		(fields_autoplaced yes)
-		(property "Reference" "#PWR018"
+		(property "Reference" "#PWR097"
 			(at 233.68 50.8 0)
 			(effects
@@
 			(project "Payload_Controller_EM"
 				(path "/866a965d-c307-40b7-9977-69e77fc0dc82/3853f2b5-b86c-4f53-9549-ed8b814cc447"
-					(reference "#PWR018")
+					(reference "#PWR097")
 					(unit 1)
 				)
@@
 		(dnp no)
 		(fields_autoplaced yes)
-		(property "Reference" "#PWR022"
+		(property "Reference" "#PWR098"
 			(at 261.62 53.34 0)
 			(effects
@@
 			(project "Payload_Controller_EM"
 				(path "/866a965d-c307-40b7-9977-69e77fc0dc82/3853f2b5-b86c-4f53-9549-ed8b814cc447"
-					(reference "#PWR022")
+					(reference "#PWR098")
 					(unit 1)
 				)
@@
 		(on_board yes)
 		(dnp no)
-		(property "Reference" "U4"
+		(property "Reference" "U8"
 			(at 126.746 107.188 0)
 			(effects
@@
 			(project "Payload_Controller_EM"
 				(path "/866a965d-c307-40b7-9977-69e77fc0dc82/3853f2b5-b86c-4f53-9549-ed8b814cc447"
-					(reference "U4")
+					(reference "U8")
 					(unit 4)
 				)
@@
 		(on_board yes)
 		(dnp no)
-		(property "Reference" "U4"
+		(property "Reference" "U8"
 			(at 247.396 43.688 0)
 			(effects
@@
 			(project "Payload_Controller_EM"
 				(path "/866a965d-c307-40b7-9977-69e77fc0dc82/3853f2b5-b86c-4f53-9549-ed8b814cc447"
-					(reference "U4")
+					(reference "U8")
 					(unit 1)
 				)
@@
 		(dnp no)
 		(fields_autoplaced yes)
-		(property "Reference" "U4"
+		(property "Reference" "U8"
 			(at 211.455 106.68 0)
 			(effects
@@
 			(project "Payload_Controller_EM"
 				(path "/866a965d-c307-40b7-9977-69e77fc0dc82/3853f2b5-b86c-4f53-9549-ed8b814cc447"
-					(reference "U4")
+					(reference "U8")
 					(unit 3)
 				)
@@
 		(dnp no)
 		(fields_autoplaced yes)
-		(property "Reference" "C3"
+		(property "Reference" "C46"
 			(at 270.51 53.3462 0)
 			(effects
@@
 			(project "Payload_Controller_EM"
 				(path "/866a965d-c307-40b7-9977-69e77fc0dc82/3853f2b5-b86c-4f53-9549-ed8b814cc447"
-					(reference "C3")
+					(reference "C46")
 					(unit 1)
 				)
@@
 		(dnp no)
 		(fields_autoplaced yes)
-		(property "Reference" "#PWR021"
+		(property "Reference" "#PWR0101"
 			(at 273.05 67.31 0)
 			(effects
@@
 			(project "Payload_Controller_EM"
 				(path "/866a965d-c307-40b7-9977-69e77fc0dc82/3853f2b5-b86c-4f53-9549-ed8b814cc447"
-					(reference "#PWR021")
+					(reference "#PWR0101")
 					(unit 1)
 				)
@@
 		(dnp no)
 		(fields_autoplaced yes)
-		(property "Reference" "U4"
+		(property "Reference" "U8"
 			(at 128.905 168.91 0)
 			(effects
@@
 		(pin "32"
 		)
-		(pin "23"
+		(pin "1"
 		)
 		(pin "23"
@@
 		(pin "13"
 		)
-		(pin "23"
-		)
-		(pin "23"
+		(pin "24"
+		)
+		(pin "30"
 		)
 		(pin "36"
@@
 		(pin "15"
 		)
-		(pin "23"
-		)
-		(pin "23"
-		)
-		(pin "23"
-		)
-		(pin "23"
+		(pin "42"
+		)
+		(pin "21"
+		)
+		(pin "44"
+		)
+		(pin "22"
 		)
 		(pin "19"
@@
 			(project "Payload_Controller_EM"
 				(path "/866a965d-c307-40b7-9977-69e77fc0dc82/3853f2b5-b86c-4f53-9549-ed8b814cc447"
-					(reference "U4")
+					(reference "U8")
 					(unit 5)
 				)
@@
 		(dnp no)
 		(fields_autoplaced yes)
-		(property "Reference" "#PWR019"
+		(property "Reference" "#PWR096"
 			(at 233.172 68.58 0)
 			(effects
@@
 			(project "Payload_Controller_EM"
 				(path "/866a965d-c307-40b7-9977-69e77fc0dc82/3853f2b5-b86c-4f53-9549-ed8b814cc447"
-					(reference "#PWR019")
+					(reference "#PWR096")
 					(unit 1)
 				)
@@
 		(dnp no)
 		(fields_autoplaced yes)
-		(property "Reference" "#PWR023"
+		(property "Reference" "#PWR099"
 			(at 261.62 67.31 0)
 			(effects
@@
 			(project "Payload_Controller_EM"
 				(path "/866a965d-c307-40b7-9977-69e77fc0dc82/3853f2b5-b86c-4f53-9549-ed8b814cc447"
-					(reference "#PWR023")
+					(reference "#PWR099")
 					(unit 1)
 				)
@@
 		(dnp no)
 		(fields_autoplaced yes)
-		(property "Reference" "C4"
+		(property "Reference" "C45"
 			(at 259.08 53.3462 0)
 			(effects
@@
 			(project "Payload_Controller_EM"
 				(path "/866a965d-c307-40b7-9977-69e77fc0dc82/3853f2b5-b86c-4f53-9549-ed8b814cc447"
-					(reference "C4")
+					(reference "C45")
 					(unit 1)
 				)
