File: _restore_backup_2026-06-10T16-12-47-721/I2C_Components.kicad_sch (KiCad schematic)
At the start: 7 parts, among them U21 P82B715DR

Commit message: Updates to inhibit
Parts:
- C91: footprint Cap_X7R_1uF:CAP_CL21_SAM -> Capacitor_SMD:C_0402_1005Metric
Changed lines of the file:
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@@
 			)
 		)
-		(property "Footprint" "Cap_X7R_1uF:CAP_CL21_SAM"
+		(property "Footprint" "Capacitor_SMD:C_0402_1005Metric"
 			(at 167.3352 76.2 0)
 			(hide yes)
