File: _restore_backup_2026-06-10T16-12-47-721/Regulator.kicad_sch (KiCad schematic)
At the start: 35 parts, among them U14 LT3652, U9 LT8612

Commit message: Updates to inhibit
Parts:
- C40: footprint Cap_X5R_10nF:CAP_X7R_0805_AVX -> Capacitor_SMD:C_0402_1005Metric
- C41: footprint Cap_X7R_1uF:CAP_CL21_SAM -> Capacitor_SMD:C_0603_1608Metric
- U14: footprint (none) -> SON45P300X300X80-13N-D
Changed lines of the file:
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@@
 	)
 	(junction
-		(at 420.37 50.8)
+		(at 184.15 328.93)
 		(diameter 0)
 		(color 0 0 0 0)
 	)
 	(junction
-		(at 273.05 331.47)
+		(at 420.37 50.8)
 		(diameter 0)
 		(color 0 0 0 0)
 	)
 	(junction
-		(at 255.27 81.28)
+		(at 273.05 331.47)
 		(diameter 0)
 		(color 0 0 0 0)
 	)
 	(junction
-		(at 184.15 328.93)
+		(at 255.27 81.28)
 		(diameter 0)
 		(color 0 0 0 0)
@@
 			)
 		)
-		(property "Footprint" ""
+		(property "Footprint" "SON45P300X300X80-13N-D"
 			(at 288.29 176.2 0)
 			(hide yes)
@@
 			)
 		)
-		(property "Footprint" "Cap_X5R_10nF:CAP_X7R_0805_AVX"
+		(property "Footprint" "Capacitor_SMD:C_0402_1005Metric"
 			(at 176.8348 317.5 0)
 			(hide yes)
@@
 			)
 		)
-		(property "Datasheet" "https://datasheets.kyocera-avx.com/KGM_X7R.pdf"
+		(property "Datasheet" ""
 			(at 177.8 321.31 0)
 			(hide yes)
@@
 			)
 		)
-		(property "Description" "https://www.digikey.com/en/products/detail/kyocera-avx/KGM21NR71H103KT/563493"
+		(property "Description" "Unpolarized capacitor"
 			(at 177.8 321.31 0)
 			(hide yes)
@@
 			)
 		)
-		(property "Footprint" "Cap_X7R_1uF:CAP_CL21_SAM"
+		(property "Footprint" "Capacitor_SMD:C_0603_1608Metric"
 			(at 183.1848 317.5 0)
 			(hide yes)
@@
 			)
 		)
-		(property "Datasheet" "https://mm.digikey.com/Volume0/opasdata/d220001/medias/docus/609/CL21B105KBFNNNE_Spec.pdf"
+		(property "Datasheet" ""
 			(at 184.15 321.31 0)
 			(hide yes)
