File: Inhibit_System.kicad_sch (KiCad schematic)
At the start: 14 parts, among them Q10 Q_NMOS, Q11 Q_NMOS, Q12 Q_NMOS, Q13 Q_NMOS, Q2 Q_NMOS, Q7 Q_NMOS, Q9 Q_NMOS, SW2 SW_SPST, SW3 SW_SPST, SW4 SW_SPST

Commit message: Updates to inhibit
Parts:
- removed Q11, Q12: Q_NMOS, symbol Device:Q_NMOS
- added BT1: Battery, symbol Device:Battery
- added Q14, Q22: Q_NMOS, symbol Device:Q_NMOS
Connections:
- net EN: now also Q14.G, Q22.G
- net Pack+: now also BT1.1 (+), Q22.D
- net Pack-: now also BT1.2 (-), Q14.D; no longer Q13.S
- net at Q7.S, Q9.D: now also Q22.S
- new net: Q13.S, Q14.S
Other:
- note added: "Must be mechanical switches that are open when depressed and normally closed when not"
- note added: "The RBF is a pin that is inserted into a switch that is either normally open or closed. Depending on if this switch is NO or NC we either remove or install the pin IE RBF or IBF"
- note removed: "Chassis - Structure of CubeSat?"
- note removed: "Make a better inhibit System"
- note removed: "what is being removed?"
- moved on the sheet: D6, D7, D8, Q13, R29, SW2, SW3, SW4

Commit message: Inhibit system
Parts:
- removed BT1: Battery, symbol Device:Battery
Connections:
- net Solar Power: no longer Q2.D
- new net Vmmpt: Q2.D
Other:
- note added: "Will need connectors that connect to switches in this area"

Commit message: Inhibit
Parts:
- added D10: 1N914, Diode_THT:D_DO-35_SOD27_P7.62mm_Horizontal, symbol Diode:1N914
Connections:
- net Solar Power: no longer names the net of D6.2 (A)
- net Solar Power: now also D10.1 (K)
- net Vmmpt renamed V_mppt
- net V_mppt: now also D10.2 (A)
Other:
- note added: "Activation inhibit: 2 Feet switches on the top 2 Feet siwtches on the bottom"
- note added: "Generic enhanced nmos for now"
- note removed: "Activation inhibit"
- note removed: "Generic enchanced nmos for now"
- note removed: "Placeholder value"
- note removed: "Potential short from Solar Power to Pack+"

Commit message: Inhibit addition
Parts:
- added J26, J27, J28, J29, J30: INHIBIT_P2, Connector_Hirose:Hirose_DF11-4DP-2DSA_2x02_P2.00mm_Vertical, symbol Connector_Generic:Conn_02x02_Odd_Even
Connections:
- net V_mppt: now also D10.1 (K), D6.2 (A)

Commit message: Footprint fixes and cleaning up
Parts:
- renumbered J26 to J16, J27 to J17, J28 to J18, J29 to J19, J30 to J20, Q22 to Q18, R29 to R28, SW2 to SW1, SW3 to SW2, SW4 to SW3

Commit message: Some Inhibit Updates/Solarcharger
Parts:
- removed SW1, SW2, SW3: SW_SPST, symbol Switch:SW_SPST
- added SW1: SW_SPDT, symbol Switch:SW_SPDT
Connections:
- net EN: now also J19.2 (Pin_2), J19.4 (Pin_4), SW1.2 (B)
- net GND: now also SW1.1 (A)
- net RBF: no longer Q10.G
- net at D6.1 (K), D8.1 (K): now also J16.1 (Pin_1), J16.3 (Pin_3)
- net at Q18.S, Q9.D: no longer Q7.S
- net at J18.1 (Pin_1): now also J17.2 (Pin_2), J17.4 (Pin_4), J18.3 (Pin_3)
- net at J18.2 (Pin_2): now also J18.4 (Pin_4), J19.1 (Pin_1), J19.3 (Pin_3)
- net at J17.1 (Pin_1): now also J16.2 (Pin_2), J16.4 (Pin_4), J17.3 (Pin_3)
- net V_mppt renamed V_mppt_i
- new net V_mppt_o: Q7.S
- no-connect marks 0 -> 1
Other:
- note added: "*I believe we can remove Q10"
- note added: "C"
- note added: "Goes back in Vin of Solar Charger to prevent V_mppt going into UNREG"
- note added: "Installation Inhibit - RBF"
- note added: "NC"
- note added: "NO"
- note added: "Negative Terminal of Battery Pack"
- note added: "Node before Vin of Solar Charger"
- note added: "Positive Terminal of Battery Pack"
- note added: "SS-5GL13"
- note removed: "Will need connectors that connect to switches in this area"
- moved on the sheet: J16, J17, J18, J19, J20, R28

Commit message: Stuff
Connections:
- net V_mppt_i: no longer D10.1 (K), D6.2 (A), Q2.D
- new net: D10.1 (K), D6.2 (A), Q2.D
Changed lines of the file:
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@@
-	)
-	(junction
-		(at 179.07 62.23)
-		(diameter 0)
-		(color 0 0 0 0)
 	)
 	(junction
@@
 		)
 		(stroke
-			(width 0)
-			(type default)
-		)
-	)
-	(wire
-		(pts
-			(xy 175.26 62.23) (xy 179.07 62.23)
-		)
-		(stroke
