File: I2C_Components.kicad_sch (KiCad schematic)
At the start: 7 parts, among them U6 P82B715DR

Commit message: Adding in Test points
Parts:
- added TP1: SDA-MCU, symbol Connector:TestPoint
- added TP2: SCL-MCU, symbol Connector:TestPoint
- added TP3: SCL-Sensor, symbol Connector:TestPoint
- added TP4: SDA-Sensor, symbol Connector:TestPoint
Connections:
- net HS_I2C1_LCL: now also TP2.1
- net HS_I2C1_LDA: now also TP1.1
- net HS_I2C1_SCL: now also TP3.1
- net HS_I2C1_SDA: now also TP4.1
- net GND renamed VSS
Other:
- moved on the sheet: R39, R8

Commit message: Updates for debug and RBF
Parts:
- renumbered C26 to C25, C27 to C26, R8 to R39, R39 to R40, R40 to R42, TP1 to TP17, TP2 to TP18, TP4 to TP19, TP3 to TP20
Other:
- moved on the sheet: TP20
Changed lines of the file:
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@@
 	)
 	(junction
+		(at 97.79 73.66)
+		(diameter 0)
+		(color 0 0 0 0)
+	)
+	(junction
 		(at 146.05 77.47)
 		(diameter 0)
@@
 		(color 0 0 0 0)
 	)
-	(junction
-		(at 97.79 73.66)
-		(diameter 0)
-		(color 0 0 0 0)
-	)
 	(wire
 		(pts
@@
 	(wire
 		(pts
-			(xy 97.79 77.47) (xy 97.79 73.66)
+			(xy 97.79 78.74) (xy 97.79 73.66)
 		)
 		(stroke
@@
 		(in_pos_files yes)
 		(dnp no)
-		(property "Reference" "#PWR0132"
+		(property "Reference" "#PWR053"
 			(at 129.54 71.12 0)
 			(hide yes)
@@
 			(project "BMS_Board_Prototype"
 				(path "/4ee99911-836b-4752-8a2d-327c8b28dc47/faab3ee8-ea24-4642-bb04-240164625363"
-					(reference "#PWR0132")
+					(reference "#PWR053")
 					(unit 1)
 				)
@@
 		(in_pos_files yes)
 		(dnp no)
-		(property "Reference" "#PWR0127"
+		(property "Reference" "#PWR051"
 			(at 83.82 62.23 0)
 			(hide yes)
@@
 			(project "BMS_Board_Prototype"
 				(path "/4ee99911-836b-4752-8a2d-327c8b28dc47/faab3ee8-ea24-4642-bb04-240164625363"
-					(reference "#PWR0127")
+					(reference "#PWR051")
 					(unit 1)
 				)
@@
 		(in_pos_files yes)
 		(dnp no)
-		(property "Reference" "#PWR0129"
+		(property "Reference" "#PWR052"
 			(at 107.95 62.23 0)
 			(hide yes)
@@
 			(project "BMS_Board_Prototype"
 				(path "/4ee99911-836b-4752-8a2d-327c8b28dc47/faab3ee8-ea24-4642-bb04-240164625363"
-					(reference "#PWR0129")
+					(reference "#PWR052")
 					(unit 1)
 				)
@@
 		(in_pos_files yes)
 		(dnp no)
-		(property "Reference" "C26"
+		(property "Reference" "C25"
 			(at 138.43 69.85 0)
 			(show_name no)
@@
 			(project "BMS_Board_Prototype"
 				(path "/4ee99911-836b-4752-8a2d-327c8b28dc47/faab3ee8-ea24-4642-bb04-240164625363"
-					(reference "C26")
+					(reference "C25")
 					(unit 1)
 				)
@@
 		(in_pos_files yes)
 		(dnp no)
-		(property "Reference" "R40"
+		(property "Reference" "R42"
 			(at 111.252 61.722 0)
 			(show_name no)
@@
 			(project "BMS_Board_Prototype"
 				(path "/4ee99911-836b-4752-8a2d-327c8b28dc47/faab3ee8-ea24-4642-bb04-240164625363"
-					(reference "R40")
+					(reference "R42")
 					(unit 1)
 				)
@@
 		(in_pos_files yes)
 		(dnp no)
-		(property "Reference" "TP2"
+		(property "Reference" "TP18"
 			(at 78.74 79.5019 0)
 			(show_name no)
@@
 			(project "BMS_Board_Prototype"
 				(path "/4ee99911-836b-4752-8a2d-327c8b28dc47/faab3ee8-ea24-4642-bb04-240164625363"
-					(reference "TP2")
+					(reference "TP18")
 					(unit 1)
 				)
@@
 		(in_pos_files yes)
 		(dnp no)
-		(property "Reference" "R8"
+		(property "Reference" "R39"
 			(at 77.47 62.23 0)
 			(show_name no)
@@
 			(project "BMS_Board_Prototype"
 				(path "/4ee99911-836b-4752-8a2d-327c8b28dc47/faab3ee8-ea24-4642-bb04-240164625363"
-					(reference "R8")
+					(reference "R39")
 					(unit 1)
 				)
@@
 		(in_pos_files yes)
 		(dnp no)
-		(property "Reference" "C27"
+		(property "Reference" "C26"
 			(at 149.86 69.85 0)
 			(show_name no)
@@
 			(project "BMS_Board_Prototype"
 				(path "/4ee99911-836b-4752-8a2d-327c8b28dc47/faab3ee8-ea24-4642-bb04-240164625363"
-					(reference "C27")
+					(reference "C26")
 					(unit 1)
 				)
@@
 		(in_pos_files yes)
 		(dnp no)
-		(property "Reference" "TP1"
+		(property "Reference" "TP17"
 			(at 73.66 64.0081 0)
 			(show_name no)
@@
 			(project "BMS_Board_Prototype"
 				(path "/4ee99911-836b-4752-8a2d-327c8b28dc47/faab3ee8-ea24-4642-bb04-240164625363"
-					(reference "TP1")
+					(reference "TP17")
 					(unit 1)
 				)
@@
 		(in_pos_files yes)
 		(dnp no)
-		(property "Reference" "#PWR077"
+		(property "Reference" "#PWR054"
 			(at 129.54 85.09 0)
 			(hide yes)
@@
 			(project "BMS_Board_Prototype"
 				(path "/4ee99911-836b-4752-8a2d-327c8b28dc47/faab3ee8-ea24-4642-bb04-240164625363"
-					(reference "#PWR077")
+					(reference "#PWR054")
 					(unit 1)
 				)
@@
 		(in_pos_files yes)
 		(dnp no)
-		(property "Reference" "#PWR078"
+		(property "Reference" "#PWR056"
 			(at 146.05 83.82 0)
 			(hide yes)
@@
 			(project "BMS_Board_Prototype"
 				(path "/4ee99911-836b-4752-8a2d-327c8b28dc47/faab3ee8-ea24-4642-bb04-240164625363"
-					(reference "#PWR078")
+					(reference "#PWR056")
 					(unit 1)
 				)
@@
 		(in_pos_files yes)
 		(dnp no)
-		(property "Reference" "TP4"
+		(property "Reference" "TP19"
 			(at 94.234 57.658 0)
 			(show_name no)
@@
 			(project "BMS_Board_Prototype"
 				(path "/4ee99911-836b-4752-8a2d-327c8b28dc47/faab3ee8-ea24-4642-bb04-240164625363"
-					(reference "TP4")
+					(reference "TP19")
 					(unit 1)
 				)
@@
 		(in_pos_files yes)
 		(dnp no)
-		(property "Reference" "#PWR0134"
+		(property "Reference" "#PWR055"
 			(at 146.05 71.12 0)
 			(hide yes)
@@
 			(project "BMS_Board_Prototype"
 				(path "/4ee99911-836b-4752-8a2d-327c8b28dc47/faab3ee8-ea24-4642-bb04-240164625363"
-					(reference "#PWR0134")
+					(reference "#PWR055")
 					(unit 1)
 				)
@@
 		(in_pos_files yes)
 		(dnp no)
-		(property "Reference" "R39"
+		(property "Reference" "R40"
 			(at 86.868 62.23 0)
 			(show_name no)
@@
 			(project "BMS_Board_Prototype"
 				(path "/4ee99911-836b-4752-8a2d-327c8b28dc47/faab3ee8-ea24-4642-bb04-240164625363"
-					(reference "R39")
+					(reference "R40")
 					(unit 1)
 				)
@@
 	(symbol
 		(lib_id "Connector:TestPoint")
-		(at 97.79 77.47 180)
+		(at 97.79 78.74 180)
 		(unit 1)
 		(body_style 1)
@@
 		(in_pos_files yes)
 		(dnp no)
-		(property "Reference" "TP3"
-			(at 96.012 82.804 0)
+		(property "Reference" "TP20"
+			(at 96.012 84.074 0)
 			(show_name no)
 			(do_not_autoplace no)
@@
 		)
 		(property "Value" "SCL-Sensor"
-			(at 92.964 84.582 0)
+			(at 92.964 85.852 0)
 			(show_name no)
 			(do_not_autoplace no)
@@
 		)
 		(property "Footprint" ""
-			(at 92.71 77.47 0)
+			(at 92.71 78.74 0)
 			(hide yes)
 			(show_name no)
@@
 		)
 		(property "Datasheet" ""
-			(at 92.71 77.47 0)
+			(at 92.71 78.74 0)
 			(hide yes)
 			(show_name no)
@@
 		)
 		(property "Description" "test point"
-			(at 97.79 77.47 0)
+			(at 97.79 78.74 0)
 			(hide yes)
 			(show_name no)
@@
 			(project "BMS_Board_Prototype"
 				(path "/4ee99911-836b-4752-8a2d-327c8b28dc47/faab3ee8-ea24-4642-bb04-240164625363"
-					(reference "TP3")
+					(reference "TP20")
 					(unit 1)
 				)

Commit message: Updates for BOM prep
Parts:
- renumbered C25 to C31, C26 to C32, R39 to R42, R40 to R43, R41 to R44, R42 to R45, U6 to U7
Changed lines of the file:
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@@
 		(in_pos_files yes)
 		(dnp no)
-		(property "Reference" "#PWR053"
+		(property "Reference" "#PWR058"
 			(at 129.54 71.12 0)
 			(hide yes)
@@
 			(project "BMS_Board_Prototype"
 				(path "/4ee99911-836b-4752-8a2d-327c8b28dc47/faab3ee8-ea24-4642-bb04-240164625363"
-					(reference "#PWR053")
+					(reference "#PWR058")
 					(unit 1)
 				)
@@
 		(in_pos_files yes)
 		(dnp no)
-		(property "Reference" "#PWR051"
+		(property "Reference" "#PWR056"
 			(at 83.82 62.23 0)
 			(hide yes)
@@
 			(project "BMS_Board_Prototype"
 				(path "/4ee99911-836b-4752-8a2d-327c8b28dc47/faab3ee8-ea24-4642-bb04-240164625363"
-					(reference "#PWR051")
+					(reference "#PWR056")
 					(unit 1)
 				)
@@
 		(in_pos_files yes)
 		(dnp no)
-		(property "Reference" "R41"
+		(property "Reference" "R44"
 			(at 100.838 61.214 0)
 			(show_name no)
@@
 			(project "BMS_Board_Prototype"
 				(path "/4ee99911-836b-4752-8a2d-327c8b28dc47/faab3ee8-ea24-4642-bb04-240164625363"
-					(reference "R41")
+					(reference "R44")
 					(unit 1)
 				)
@@
 		(in_pos_files yes)
 		(dnp no)
-		(property "Reference" "#PWR052"
+		(property "Reference" "#PWR057"
 			(at 107.95 62.23 0)
 			(hide yes)
@@
 			(project "BMS_Board_Prototype"
 				(path "/4ee99911-836b-4752-8a2d-327c8b28dc47/faab3ee8-ea24-4642-bb04-240164625363"
-					(reference "#PWR052")
+					(reference "#PWR057")
 					(unit 1)
 				)
@@
 		(in_pos_files yes)
 		(dnp no)
-		(property "Reference" "C25"
+		(property "Reference" "C31"
 			(at 138.43 69.85 0)
 			(show_name no)
@@
 			(project "BMS_Board_Prototype"
 				(path "/4ee99911-836b-4752-8a2d-327c8b28dc47/faab3ee8-ea24-4642-bb04-240164625363"
-					(reference "C25")
+					(reference "C31")
 					(unit 1)
 				)
@@
 		(in_pos_files yes)
 		(dnp no)
-		(property "Reference" "R42"
+		(property "Reference" "R45"
 			(at 111.252 61.722 0)
 			(show_name no)
@@
 			(project "BMS_Board_Prototype"
 				(path "/4ee99911-836b-4752-8a2d-327c8b28dc47/faab3ee8-ea24-4642-bb04-240164625363"
-					(reference "R42")
+					(reference "R45")
 					(unit 1)
 				)
@@
 		(in_pos_files yes)
 		(dnp no)
-		(property "Reference" "U6"
+		(property "Reference" "U7"
 			(at 120.904 81.534 0)
 			(show_name no)
@@
 			(project "BMS_Board_Prototype"
 				(path "/4ee99911-836b-4752-8a2d-327c8b28dc47/faab3ee8-ea24-4642-bb04-240164625363"
-					(reference "U6")
+					(reference "U7")
 					(unit 1)
 				)
@@
 		(in_pos_files yes)
 		(dnp no)
-		(property "Reference" "R39"
+		(property "Reference" "R42"
 			(at 77.47 62.23 0)
 			(show_name no)
@@
 			(project "BMS_Board_Prototype"
 				(path "/4ee99911-836b-4752-8a2d-327c8b28dc47/faab3ee8-ea24-4642-bb04-240164625363"
-					(reference "R39")
+					(reference "R42")
 					(unit 1)
 				)
@@
 		(in_pos_files yes)
 		(dnp no)
-		(property "Reference" "C26"
+		(property "Reference" "C32"
 			(at 149.86 69.85 0)
 			(show_name no)
@@
 			(project "BMS_Board_Prototype"
 				(path "/4ee99911-836b-4752-8a2d-327c8b28dc47/faab3ee8-ea24-4642-bb04-240164625363"
-					(reference "C26")
+					(reference "C32")
 					(unit 1)
 				)
@@
 		(in_pos_files yes)
 		(dnp no)
-		(property "Reference" "#PWR054"
+		(property "Reference" "#PWR059"
 			(at 129.54 85.09 0)
 			(hide yes)
@@
 			(project "BMS_Board_Prototype"
 				(path "/4ee99911-836b-4752-8a2d-327c8b28dc47/faab3ee8-ea24-4642-bb04-240164625363"
-					(reference "#PWR054")
+					(reference "#PWR059")
 					(unit 1)
 				)
@@
 		(in_pos_files yes)
 		(dnp no)
-		(property "Reference" "#PWR056"
+		(property "Reference" "#PWR061"
 			(at 146.05 83.82 0)
 			(hide yes)
@@
 			(project "BMS_Board_Prototype"
 				(path "/4ee99911-836b-4752-8a2d-327c8b28dc47/faab3ee8-ea24-4642-bb04-240164625363"
-					(reference "#PWR056")
+					(reference "#PWR061")
 					(unit 1)
 				)
@@
 		(in_pos_files yes)
 		(dnp no)
-		(property "Reference" "#PWR055"
+		(property "Reference" "#PWR060"
 			(at 146.05 71.12 0)
 			(hide yes)
@@
 			(project "BMS_Board_Prototype"
 				(path "/4ee99911-836b-4752-8a2d-327c8b28dc47/faab3ee8-ea24-4642-bb04-240164625363"
-					(reference "#PWR055")
+					(reference "#PWR060")
 					(unit 1)
 				)
@@
 		(in_pos_files yes)
 		(dnp no)
-		(property "Reference" "R40"
+		(property "Reference" "R43"
 			(at 86.868 62.23 0)
 			(show_name no)
@@
 			(project "BMS_Board_Prototype"
 				(path "/4ee99911-836b-4752-8a2d-327c8b28dc47/faab3ee8-ea24-4642-bb04-240164625363"
-					(reference "R40")
-					(unit 1)
-				)
+					(reference "R43")
+					(unit 1)
+				)

Commit message: Adding in EMI and GND ties
Connections:
- net +3.3V: no longer R42.1, R43.1, R44.1, R45.1
- new net +3.3V Q: R42.1, R43.1, R44.1, R45.1
Changed lines of the file:
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@@
 			)
 		)
-		(property "Value" "+3.3V"
+		(property "Value" "+3.3V Q"
 			(at 83.82 54.61 0)
 			(show_name no)
@@
 			)
 		)
-		(property "Value" "+3.3V"
+		(property "Value" "+3.3V Q"
 			(at 107.95 54.61 0)
 			(show_name no)
