File: I2C_Components.kicad_sch (KiCad schematic)
At the start: 11 parts, among them U7 P82B715DR

Commit message: Updates to footprints for PCB
Parts:
- C31: footprint Cap_X7R_1uF:CAP_CL21_SAM -> Capacitor_SMD:C_0805_2012Metric
- R42, R43, R44, R45: footprint (none) -> Resistor_SMD:R_0805_2012Metric
- U7: footprint Footprints:SOIC127P600X175-8N -> I2C_buffer:D8
Changed lines of the file:
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@@
 			)
 		)
-		(property "Footprint" ""
+		(property "Footprint" "Resistor_SMD:R_0805_2012Metric"
 			(at 104.902 63.5 90)
 			(hide yes)
@@
 			)
 		)
-		(property "Footprint" "Cap_X7R_1uF:CAP_CL21_SAM"
+		(property "Footprint" "Capacitor_SMD:C_0805_2012Metric"
 			(at 143.2052 76.2 0)
 			(hide yes)
@@
 			)
 		)
-		(property "Footprint" ""
+		(property "Footprint" "Resistor_SMD:R_0805_2012Metric"
 			(at 107.442 63.5 90)
 			(hide yes)
@@
 			)
 		)
-		(property "Footprint" "Footprints:SOIC127P600X175-8N"
+		(property "Footprint" "I2C_buffer:D8"
 			(at 120.65 64.77 0)
 			(hide yes)
@@
 			)
 		)
-		(property "Footprint" ""
+		(property "Footprint" "Resistor_SMD:R_0805_2012Metric"
 			(at 80.772 63.5 90)
 			(hide yes)
@@
 			)
 		)
-		(property "Footprint" ""
+		(property "Footprint" "Resistor_SMD:R_0805_2012Metric"
 			(at 83.312 63.5 90)
 			(hide yes)

Commit message: Starting PCB layout and checking footprints
Parts:
- TP17, TP18, TP19, TP20: footprint (none) -> TestPoint:TestPoint_THTPad_D1.0mm_Drill0.5mm
Changed lines of the file:
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@@
 			)
 		)
-		(property "Footprint" ""
+		(property "Footprint" "TestPoint:TestPoint_THTPad_D1.0mm_Drill0.5mm"
 			(at 71.12 77.47 0)
 			(hide yes)
@@
 			)
 		)
-		(property "Footprint" ""
+		(property "Footprint" "TestPoint:TestPoint_THTPad_D1.0mm_Drill0.5mm"
 			(at 81.28 66.04 0)
 			(hide yes)
@@
 			)
 		)
-		(property "Footprint" ""
+		(property "Footprint" "TestPoint:TestPoint_THTPad_D1.0mm_Drill0.5mm"
 			(at 102.87 64.77 0)
 			(hide yes)
@@
 			)
 		)
-		(property "Footprint" ""
+		(property "Footprint" "TestPoint:TestPoint_THTPad_D1.0mm_Drill0.5mm"
 			(at 92.71 78.74 0)
 			(hide yes)

Commit message: PCB/Schematic updates
Connections:
- net +3.3V is gone; now on net +3.3V Q: C31.1, C32.1, U7.8 (Vcc)
Changed lines of the file:
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@@
 			)
 		)
-		(property "Value" "+3.3V"
+		(property "Value" "+3.3V Q"
 			(at 129.54 63.5 0)
 			(show_name no)
@@
 			)
 		)
-		(property "Value" "+3.3V"
+		(property "Value" "+3.3V Q"
 			(at 146.05 63.5 0)
 			(show_name no)

Commit message: Forgot to save :(
Parts:
- C31: footprint Capacitor_SMD:C_0805_2012Metric -> Resistor_SMD:R_0603_1608Metric
- C32: footprint Capacitor_SMD:C_0402_1005Metric -> Resistor_SMD:R_0603_1608Metric
Changed lines of the file:
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@@
 			)
 		)
-		(property "Footprint" "Capacitor_SMD:C_0805_2012Metric"
+		(property "Footprint" "Resistor_SMD:R_0603_1608Metric"
 			(at 143.2052 76.2 0)
 			(hide yes)
@@
 			)
 		)
-		(property "Footprint" "Capacitor_SMD:C_0402_1005Metric"
+		(property "Footprint" "Resistor_SMD:R_0603_1608Metric"
 			(at 150.8252 76.2 0)
 			(hide yes)
